Commit message: modify the urdf without mesh for the real robot

File: niryo_robot_description/urdf/ned/without_mesh_niryo_ned.urdf.xacro (robot description, xacro)
@@ -94,4 +94,22 @@
         </collision>
     </link>
+    <!-- Test to add collision for the motor of joint 5 -->
+    <link name="test_collision">
+        <collision>
+            <origin xyz="-0.045 0.0 0.1765"
+                    rpy="0 0 0"/>
+            <geometry>
+                <box size="0.034 0.0285 0.0465"/>
+            </geometry>
+        </collision>
+    </link>
+    <joint name="joint_test"
+           type="fixed">
+        <origin xyz="0 0 0"
+                rpy="0 0 0"/>
+        <parent link="forearm_link"/>
+        <child link="test_collision"/>
+    </joint>
+    <!-- end of test -->
     <joint name="joint_5"
            type="revolute">
