Commit message: add collision for joint 5 motor

File: niryo_robot_description/urdf/ned/niryo_ned.urdf.xacro (robot description, xacro)
@@ -159,4 +159,28 @@
         </collision>
     </link>
+    <!-- Test to add collision for the motor of joint 5 -->
+    <link name="test_collision">
+        <inertial>
+            <origin xyz="-0.00811345462189901 -0.000135618649565461 0.107402242790047"
+                    rpy="0 0 0"/>
+            <mass value="0.203543862275952"/>
+            <inertia ixx="0.0015" ixy="0.0" ixz="0.0" iyy="0.0015" iyz="0.0" izz="0.0015"/>
+        </inertial>
+        <collision>
+            <origin xyz="-0.045 0.0 0.1765"
+                    rpy="0 0 0"/>
+            <geometry>
+                <box size="0.03 0.03 0.046"/> <!-- le y et le z sont inverse -->
+            </geometry>
+        </collision>
+    </link>
+    <joint name="joint_test"
+           type="fixed">
+        <origin xyz="0 0 0"
+                rpy="0 0 0"/>
+        <parent link="forearm_link"/>
+        <child link="test_collision"/>
+    </joint>
+    <!-- end of test -->
     <joint name="joint_5"
            type="revolute">

Commit message: clean urdf

File: niryo_robot_description/urdf/ned/niryo_ned.urdf.xacro (robot description, xacro)
@@ -159,6 +159,6 @@
         </collision>
     </link>
-    <!-- Test to add collision for the motor of joint 5 -->
-    <link name="test_collision">
+    <!-- add collision for the motor of joint 5 -->
+    <link name="joint5_motor">
         <inertial>
             <origin xyz="-0.00811345462189901 -0.000135618649565461 0.107402242790047"
@@ -180,7 +180,6 @@
                 rpy="0 0 0"/>
         <parent link="forearm_link"/>
-        <child link="test_collision"/>
-    </joint>
-    <!-- end of test -->
+        <child link="joint5_motor"/>
+    </joint>
     <joint name="joint_5"
            type="revolute">

File: niryo_robot_description/urdf/ned/without_mesh_niryo_ned.urdf.xacro (robot description, xacro)
@@ -94,6 +94,6 @@
         </collision>
     </link>
-    <!-- Test to add collision for the motor of joint 5 -->
-    <link name="test_collision">
+    <!-- add collision for the motor of joint 5 -->
+    <link name="joint5_motor">
         <collision>
             <origin xyz="-0.045 0.0 0.1765"
@@ -109,7 +109,6 @@
                 rpy="0 0 0"/>
         <parent link="forearm_link"/>
-        <child link="test_collision"/>
+        <child link="joint5_motor"/>
     </joint>
-    <!-- end of test -->
     <joint name="joint_5"
            type="revolute">

Commit message: update box size to be bigger than motor 5

File: niryo_robot_description/urdf/ned/niryo_ned.urdf.xacro (robot description, xacro)
@@ -171,5 +171,6 @@
                     rpy="0 0 0"/>
             <geometry>
-                <box size="0.03 0.03 0.046"/> <!-- le y et le z sont inverse -->
+                <!-- <box size="0.03 0.03 0.046"/>  -->
+                <box size="0.0435 0.0285 0.0465"/>
             </geometry>
         </collision>

File: niryo_robot_description/urdf/ned/without_mesh_niryo_ned.urdf.xacro (robot description, xacro)
@@ -100,5 +100,5 @@
                     rpy="0 0 0"/>
             <geometry>
-                <box size="0.034 0.0285 0.0465"/>
+                <box size="0.0435 0.0285 0.0465"/>
             </geometry>
         </collision>

Commit message: Fix one simu limits

File: niryo_robot_description/urdf/ned/niryo_ned.urdf.xacro (robot description, xacro)
@@ -32,4 +32,5 @@
         </collision>
     </link>
+    <!--Joints -->
     <joint name="joint_1"
            type="revolute">

File: niryo_robot_description/urdf/ned/niryo_ned_param.urdf.xacro (robot description, xacro)
@@ -7,14 +7,14 @@
     <xacro:property name="limit_low_shoulder_rotation" value="-170.0"/>
     <xacro:property name="limit_up_shoulder_rotation" value="170.0"/>
-    <xacro:property name="limit_low_arm_rotation" value="-120.0"/>
-    <xacro:property name="limit_up_arm_rotation" value="35.0"/>
-    <xacro:property name="limit_low_elbow_rotation" value="-77.0"/>
-    <xacro:property name="limit_up_elbow_rotation" value="90.0"/>
-    <xacro:property name="limit_low_forearm_rotation" value="-120.0"/>
-    <xacro:property name="limit_up_forearm_rotation" value="120.0"/>
-    <xacro:property name="limit_low_wrist_rotation" value="-120.0"/>
-    <xacro:property name="limit_up_wrist_rotation" value="60.0"/>
-    <xacro:property name="limit_low_hand_rotation" value="-145.0"/>
-    <xacro:property name="limit_up_hand_rotation" value="145.0"/>
+    <xacro:property name="limit_low_arm_rotation" value="-119.75"/>
+    <xacro:property name="limit_up_arm_rotation" value="34.96"/>
+    <xacro:property name="limit_low_elbow_rotation" value="-76.78"/>
+    <xacro:property name="limit_up_elbow_rotation" value="89.96"/>
+    <xacro:property name="limit_low_forearm_rotation" value="-119.75"/>
+    <xacro:property name="limit_up_forearm_rotation" value="119.75"/>
+    <xacro:property name="limit_low_wrist_rotation" value="-110.01"/>
+    <xacro:property name="limit_up_wrist_rotation" value="60.17"/>
+    <xacro:property name="limit_low_hand_rotation" value="-144.96"/>
+    <xacro:property name="limit_up_hand_rotation" value="144.96"/>
     <xacro:property name="safety_pos_margin" value="0.0"/>
 </robot>

File: niryo_robot_description/urdf/ned2/niryo_ned2_param.urdf.xacro (robot description, xacro)
@@ -5,16 +5,16 @@
     <!-- Properties -->
     <xacro:property name="distance_hand_tool" value="0.0215"/>
-    <xacro:property name="limit_low_shoulder_rotation" value="-169.0"/>
-    <xacro:property name="limit_up_shoulder_rotation" value="169.0"/>
-    <xacro:property name="limit_low_arm_rotation" value="-120.0"/>
-    <xacro:property name="limit_up_arm_rotation" value="35.0"/>
-    <xacro:property name="limit_low_elbow_rotation" value="-77.0"/>
-    <xacro:property name="limit_up_elbow_rotation" value="90.0"/>
-    <xacro:property name="limit_low_forearm_rotation" value="-120.0"/>
-    <xacro:property name="limit_up_forearm_rotation" value="120.0"/>
-    <xacro:property name="limit_low_wrist_rotation" value="-110.0"/>
-    <xacro:property name="limit_up_wrist_rotation" value="110.0"/>
-    <xacro:property name="limit_low_hand_rotation" value="-145.0"/>
-    <xacro:property name="limit_up_hand_rotation" value="145.0"/>
+    <xacro:property name="limit_low_shoulder_rotation" value="-169.03"/>
+    <xacro:property name="limit_up_shoulder_rotation" value="169.03"/>
+    <xacro:property name="limit_low_arm_rotation" value="-119.75"/>
+    <xacro:property name="limit_up_arm_rotation" value="34.96"/>
+    <xacro:property name="limit_low_elbow_rotation" value="-76.78"/>
+    <xacro:property name="limit_up_elbow_rotation" value="89.96"/>
+    <xacro:property name="limit_low_forearm_rotation" value="-119.75"/>
+    <xacro:property name="limit_up_forearm_rotation" value="119.75"/>
+    <xacro:property name="limit_low_wrist_rotation" value="-110.01"/>
+    <xacro:property name="limit_up_wrist_rotation" value="60.17"/>
+    <xacro:property name="limit_low_hand_rotation" value="-144.96"/>
+    <xacro:property name="limit_up_hand_rotation" value="144.96"/>
     <xacro:property name="safety_pos_margin" value="0.0"/>
 </robot>

File: niryo_robot_description/urdf/one/niryo_one.urdf.xacro (robot description, xacro)
@@ -160,6 +160,6 @@
         <origin xyz="0 0 ${distance_origin_shoulder_z}" rpy="0 0 0"/>
         <axis xyz="0 0 1"/>
-        <limit effort="10.0" velocity="2.2" lower="${limit_low_shoulder_rotation}"
-               upper="${limit_up_shoulder_rotation}"/>
+        <limit effort="10.0" velocity="2.2" lower="${(limit_low_shoulder_rotation + safety_pos_margin) * deg_to_rad}"
+               upper="${(limit_up_shoulder_rotation - safety_pos_margin) * deg_to_rad}"/>
         <dynamics damping="0.1" friction="0.0"/>
     </joint>
@@ -168,5 +168,6 @@
         <child link="arm_link"/>
         <origin xyz="0 0 ${distance_shoulder_arm_z}" rpy="${PI/2} ${-PI/2} 0"/>
-        <limit effort="10.0" velocity="2.2" lower="${limit_low_arm_rotation}" upper="${limit_up_arm_rotation}"/>
+        <limit effort="10.0" velocity="2.2" lower="${(limit_low_arm_rotation + safety_pos_margin) * deg_to_rad}"
+               upper="${(limit_up_arm_rotation - safety_pos_margin) * deg_to_rad}"/>
         <axis xyz="0 0 1"/>
         <dynamics damping="0.1" friction="0.0"/>
@@ -176,5 +177,6 @@
         <child link="elbow_link"/>
         <origin xyz="${distance_arm_elbow_x} ${distance_arm_elbow_y} 0" rpy="0 0 ${-PI/2}"/>
-        <limit effort="7.0" velocity="2.0" lower="${limit_low_elbow_rotation}" upper="${limit_up_elbow_rotation}"/>
+        <limit effort="7.0" velocity="2.0" lower="${(limit_low_elbow_rotation + safety_pos_margin) * deg_to_rad}"
+               upper="${(limit_up_elbow_rotation - safety_pos_margin) * deg_to_rad}"/>
         <axis xyz="0 0 1"/>
         <dynamics damping="0.1" friction="0.0"/>
@@ -184,6 +186,6 @@
         <child link="forearm_link"/>
         <origin xyz="${distance_elbow_forearm_x} ${distance_elbow_forearm_y} 0" rpy="0 ${PI/2} 0"/>
-        <limit effort="7.0" velocity="2.0" lower="${limit_low_forearm_rotation}"
-               upper="${limit_up_forearm_rotation}"/>
+        <limit effort="7.0" velocity="2.0" lower="${(limit_low_forearm_rotation + safety_pos_margin) * deg_to_rad}"
+               upper="${(limit_up_forearm_rotation - safety_pos_margin) * deg_to_rad}"/>
         <axis xyz="0 0 1"/>
         <dynamics damping="0.1" friction="0.0"/>
@@ -193,5 +195,6 @@
         <child link="wrist_link"/>
         <origin xyz="0 0 ${distance_forearm_wrist_z}" rpy="0 ${-PI/2} 0"/>
-        <limit effort="6.0" velocity="2.0" lower="${limit_low_wrist_rotation}" upper="${limit_up_wrist_rotation}"/>
+        <limit effort="6.0" velocity="2.0" lower="${(limit_low_wrist_rotation + safety_pos_margin) * deg_to_rad}"
+               upper="${(limit_up_wrist_rotation - safety_pos_margin) * deg_to_rad}"/>
         <axis xyz="0 0 1"/>
         <dynamics damping="0.1" friction="0.0"/>
@@ -201,5 +204,6 @@
         <child link="hand_link"/>
         <origin xyz="${distance_wrist_hand_x} ${distance_wrist_hand_y} 0" rpy="0 ${PI/2} 0"/>
-        <limit effort="5.0" velocity="2.0" lower="${limit_low_hand_rotation}" upper="${limit_up_hand_rotation}"/>
+        <limit effort="5.0" velocity="2.0" lower="${(limit_low_hand_rotation + safety_pos_margin) * deg_to_rad}"
+               upper="${(limit_up_hand_rotation - safety_pos_margin) * deg_to_rad}"/>
         <axis xyz="0 0 1"/>
         <dynamics damping="0.1" friction="0.0"/>

File: niryo_robot_description/urdf/one/niryo_one_param.urdf.xacro (robot description, xacro)
@@ -14,15 +14,16 @@
     <xacro:property name="distance_wrist_hand_y" value="-0.0055" />
     <xacro:property name="distance_hand_tool" value="0.0073" />
-    <xacro:property name="limit_low_shoulder_rotation" value="-3.05433" />
-    <xacro:property name="limit_up_shoulder_rotation" value="3.05433" />
-    <xacro:property name="limit_low_arm_rotation" value="-1.91986" />
-    <xacro:property name="limit_up_arm_rotation" value="0.640187" />
-    <xacro:property name="limit_low_elbow_rotation" value="-1.397485" />
-    <xacro:property name="limit_up_elbow_rotation" value="${PI/2}" />
-    <xacro:property name="limit_low_forearm_rotation" value="-3.05433" />
-    <xacro:property name="limit_up_forearm_rotation" value="3.05433" />
-    <xacro:property name="limit_low_wrist_rotation" value="-1.74533" />
-    <xacro:property name="limit_up_wrist_rotation" value="1.91986" />
-    <xacro:property name="limit_low_hand_rotation" value="-2.57436" />
-    <xacro:property name="limit_up_hand_rotation" value="2.57436" />
+    <xacro:property name="limit_low_shoulder_rotation" value="-175.0" />
+    <xacro:property name="limit_up_shoulder_rotation" value="175.0" />
+    <xacro:property name="limit_low_arm_rotation" value="-109.44" />
+    <xacro:property name="limit_up_arm_rotation" value="36.67" />
+    <xacro:property name="limit_low_elbow_rotation" value="-79.89" />
+    <xacro:property name="limit_up_elbow_rotation" value="89.96" />
+    <xacro:property name="limit_low_forearm_rotation" value="-174.76" />
+    <xacro:property name="limit_up_forearm_rotation" value="175.0" />
+    <xacro:property name="limit_low_wrist_rotation" value="-100.0" />
+    <xacro:property name="limit_up_wrist_rotation" value="110.01" />
+    <xacro:property name="limit_low_hand_rotation" value="-144.96" />
+    <xacro:property name="limit_up_hand_rotation" value="144.96" />
+    <xacro:property name="safety_pos_margin" value="0.0"/>
 </robot>
