Commit message: Increasing the limits of the joint5 for the vision kit

File: niryo_robot_description/urdf/ned/niryo_ned_param.urdf.xacro (robot description, xacro)
@@ -12,6 +12,6 @@
     <xacro:property name="limit_low_forearm_rotation" value="-120.0"/>
     <xacro:property name="limit_up_forearm_rotation" value="120.0"/>
-    <xacro:property name="limit_low_wrist_rotation" value="-100.0"/>
-    <xacro:property name="limit_up_wrist_rotation" value="55.0"/>
+    <xacro:property name="limit_low_wrist_rotation" value="-120.0"/>
+    <xacro:property name="limit_up_wrist_rotation" value="60.0"/>
     <xacro:property name="limit_low_hand_rotation" value="-145.0"/>
     <xacro:property name="limit_up_hand_rotation" value="145.0"/>

Commit message: beta3-v4.1.0

File: niryo_robot_description/urdf/ned/niryo_ned_param.urdf.xacro (robot description, xacro)
@@ -7,5 +7,5 @@
     <xacro:property name="limit_low_shoulder_rotation" value="-170.0"/>
     <xacro:property name="limit_up_shoulder_rotation" value="170.0"/>
-    <xacro:property name="limit_low_arm_rotation" value="-119.75"/>
+    <xacro:property name="limit_low_arm_rotation" value="-109.44"/>
     <xacro:property name="limit_up_arm_rotation" value="34.96"/>
     <xacro:property name="limit_low_elbow_rotation" value="-76.78"/>

File: niryo_robot_description/urdf/ned2/niryo_ned2.urdf.xacro (robot description, xacro)
@@ -61,12 +61,10 @@
     <link name="arm_link">
         <inertial>
-            <origin xyz="0.116485160625991 -0.00141190194997476 -0.00338105503061108"
-                    rpy="0 0 0"/>
-            <mass value="0.513332159226246"/>
-            <inertia ixx="0.0015" ixy="0.0" ixz="0.0" iyy="0.0015" iyz="0.0" izz="0.0015"/>
-        </inertial>
-        <visual>
-            <origin xyz="0 0 0"
-                    rpy="0 0 0"/>
+            <origin xyz="-0.00096976 0.086432 0.0038832" rpy="0 ${PI} 0"/>
+            <mass value="1.0838"/>
+            <inertia ixx="0.008194" ixy="0.00015602" ixz="-3.434E-06" iyy="0.0011945" iyz="-0.00031298" izz="0.007915"/>
+        </inertial>
+        <visual>
+            <origin xyz="0 0 0" rpy="0 ${PI} 0"/>
             <geometry>
                 <mesh filename="package://niryo_robot_description/meshes/ned2/collada/arm_link.dae"/>
@@ -74,6 +72,5 @@
         </visual>
         <collision>
-            <origin xyz="0 0 0"
-                    rpy="0 0 0"/>
+            <origin xyz="0 0 0" rpy="0 ${PI} 0"/>
             <geometry>
                 <mesh filename="package://niryo_robot_description/meshes/ned2/stl/arm_link.stl"/>
@@ -83,13 +80,11 @@
     <link name="elbow_link">
         <inertial>
-            <origin
-                    xyz="0.0082004 0.023746 0.0053676" rpy="0 0 0"/>
-            <mass value="0.15494"/>
-            <inertia ixx="6.0879E-05" ixy="-1.2086E-05" ixz="-1.3026E-08" iyy="7.4479E-05" iyz="-4.6729E-08"
-                     izz="9.8727E-05"/>
-        </inertial>
-        <visual>
-            <origin xyz="0 0 0"
-                    rpy="0 0 0"/>
+            <origin xyz="-0.019703 0.037336 -1.7431E-09" rpy="0 ${PI} 0"/>
+            <mass value="0.22126"/>
+            <inertia ixx="0.00011754" ixy="-1.2314E-05" ixz="-6.2064E-11" iyy="0.00020851" iyz="9.2393E-11"
+                     izz="0.00022753"/>
+        </inertial>
+        <visual>
+            <origin xyz="0 0 0" rpy="0 ${PI} 0"/>
             <geometry>
                 <mesh filename="package://niryo_robot_description/meshes/ned2/collada/elbow_link.dae"/>
@@ -97,6 +92,5 @@
         </visual>
         <collision>
-            <origin xyz="0 0 0"
-                    rpy="0 0 0"/>
+            <origin xyz="0 0 0" rpy="0 ${PI} 0"/>
             <geometry>
                 <mesh filename="package://niryo_robot_description/meshes/ned2/stl/elbow_link.stl"/>
@@ -106,8 +100,8 @@
     <link name="forearm_link">
         <inertial>
-            <origin xyz="-0.0094603 8.5954E-05 0.10662" rpy="0 0 0"/>
-            <mass value="0.16445"/>
-            <inertia ixx="0.00015109" ixy="-1.6205E-07" ixz="4.3654E-07" iyy="0.00014456" iyz="-3.9296E-07"
-                     izz="4.8807E-05"/>
+            <origin xyz="-0.0049532 7.8351E-06 0.08106" rpy="0 0 0"/>
+            <mass value="0.35686"/>
+            <inertia ixx="0.0013664" ixy="-9.6367E-08" ixz="0.00013594" iyy="0.0014781" iyz="-1.4596E-07"
+                     izz="0.00023715"/>
         </inertial>
         <visual>
@@ -124,5 +118,5 @@
         </collision>
     </link>
-    <!-- add collision for the motor of joint 5 -->
+    <!-- add collision for the motor of joint 5
     <link name="joint5_motor">
         <inertial>
@@ -137,11 +131,10 @@
             </geometry>
         </collision>
-    </link>
+    </link> -->
     <link name="wrist_link">
         <inertial>
-            <origin xyz="-0.020082 0.0015621 9.3782E-05" rpy="0 0 0"/>
-            <mass value="0.03067"/>
-            <inertia ixx="4.2466E-06" ixy="-2.9761E-07" ixz="-9.1198E-09" iyy="3.6068E-06" iyz="-3.5847E-08"
-                     izz="3.801E-06"/>
+            <origin xyz="-0.019666 0.037312 0.0" rpy="0 0 0"/>
+            <mass value="0.22126"/>
+            <inertia ixx="0.0015" ixy="0.0" ixz="0.0" iyy="0.0015" iyz="0.0" izz="0.0015"/>
         </inertial>
         <visual>
@@ -188,5 +181,5 @@
     </joint>
     <joint name="joint_1" type="revolute">
-        <origin xyz="0 3.7961E-05 0.1013" rpy="0 0 0"/>
+        <origin xyz="0 0 0.1013" rpy="0 0 ${-PI/2}"/>
         <parent link="base_link"/>
         <child link="shoulder_link"/>
@@ -196,5 +189,5 @@
     </joint>
     <joint name="joint_2" type="revolute">
-        <origin xyz="0 0 0.065" rpy="${PI/2} ${-PI/2} 0"/>
+        <origin xyz="0 0 0.065" rpy="${PI/2} 0 ${PI/2}"/>
         <parent link="shoulder_link"/>
         <child link="arm_link"/>
@@ -204,5 +197,5 @@
     </joint>
     <joint name="joint_3" type="revolute">
-        <origin xyz="0.221 -0.012 0" rpy="0 0 ${-PI/2}"/>
+        <origin xyz="0.012 0.221 0" rpy="0 0 0"/>
         <parent link="arm_link"/>
         <child link="elbow_link"/>
@@ -240,9 +233,10 @@
         <origin xyz="0 0 ${distance_hand_tool}" rpy="${-PI/2} ${-PI/2} 0"/>
     </joint>
+    <!--
     <joint name="joint_test" type="fixed">
         <origin xyz="-0.03 0 0.158" rpy="0 -${PI/2} 0"/>
         <parent link="forearm_link"/>
         <child link="joint5_motor"/>
-    </joint>
+    </joint> -->
     <joint name="joint_led_ring" type="fixed">
         <parent link="world"/>

File: niryo_robot_description/urdf/ned2/niryo_ned2_gripper1_n_camera.urdf.xacro (robot description, xacro)
@@ -4,5 +4,5 @@
     <!-- gazebo joint state publisher for all joints. Necessary to control mors -->
     <gazebo>
-        <plugin name="passive_joint_state_publisher" filename="libgazebo_ros_joint_state_publisher.so">
+        <plugin name="joint_state_publisher" filename="libgazebo_ros_joint_state_publisher.so">
             <jointName>joint_1, joint_2, joint_3, joint_4, joint_5, joint_6,
                 joint_base_to_mors_1, joint_base_to_mors_2
@@ -17,6 +17,6 @@
         <child link="base_gripper_1"/>
         <origin
-                xyz="0.005 0 0.005"
-                rpy="0 ${PI/2} ${PI/2}"/>
+                xyz="0.003 0 -0.007"
+                rpy="0 ${-PI/2} ${PI/2}"/>
     </joint>
     <!-- Base Gripper -->

File: niryo_robot_description/urdf/ned2/niryo_ned2_param.urdf.xacro (robot description, xacro)
@@ -4,8 +4,8 @@
     <xacro:property name="deg_to_rad" value="${PI/180}"/>
     <!-- Properties -->
-    <xacro:property name="distance_hand_tool" value="0.0215"/>
+    <xacro:property name="distance_hand_tool" value="0.0285"/>
     <xacro:property name="limit_low_shoulder_rotation" value="-169.03"/>
     <xacro:property name="limit_up_shoulder_rotation" value="169.03"/>
-    <xacro:property name="limit_low_arm_rotation" value="-119.75"/>
+    <xacro:property name="limit_low_arm_rotation" value="-105.0"/>
     <xacro:property name="limit_up_arm_rotation" value="34.96"/>
     <xacro:property name="limit_low_elbow_rotation" value="-76.78"/>

File: niryo_robot_description/urdf/ned2/without_mesh_niryo_ned2.urdf.xacro (robot description, xacro)
@@ -6,64 +6,123 @@
     <link name="world"/>
     <link name="base_link">
+        <inertial>
+            <origin xyz="-0.008924 0.0001357 0.052392" rpy="0 0 0"/>
+            <mass value="0.71142"/>
+            <inertia ixx="0.0017" ixy="0.0" ixz="0.0" iyy="0.0017" iyz="0.0" izz="0.0032"/>
+        </inertial>
+        <collision>
+            <origin xyz="0 0 0" rpy="-${PI/2} 0 0"/>
+            <geometry>
+                <mesh filename="package://niryo_robot_description/meshes/ned2/stl/base_link.stl"/>
+            </geometry>
+        </collision>
+    </link>
+    <link name="led_ring_link">
+        <!--
+        <visual>
+            <origin xyz="0 0 0"
+                    rpy="0 0 0"/>
+            <geometry>
+                <cylinder length="0.0019" radius="0.0775"/>
+            </geometry>
+            <material
+                    name="">
+                <color
+                        rgba="1 1 1 0.25"/>
+            </material>
+        </visual> -->
+    </link>
+    <link name="shoulder_link">
+        <inertial>
+            <origin xyz="-0.031951 0.0080419 0.030675" rpy="0 0 0"/>
+            <mass value="0.35056"/>
+            <inertia ixx="0.00023875" ixy="2.3853E-08" ixz="2.0596E-06" iyy="0.00032638" iyz="-8.9319E-07"
+                     izz="0.00030089"/>
+        </inertial>
         <collision>
             <origin xyz="0 0 0" rpy="0 0 0"/>
             <geometry>
-                <mesh filename="package://niryo_robot_description/meshes/ned2/stl/base_link.stl"/>
-            </geometry>
-        </collision>
-    </link>
-    <link name="shoulder_link">
+                <mesh filename="package://niryo_robot_description/meshes/ned2/stl/shoulder_link.stl"/>
+            </geometry>
+        </collision>
+    </link>
+    <link name="arm_link">
+        <inertial>
+            <origin xyz="-0.00096976 0.086432 0.0038832" rpy="0 ${PI} 0"/>
+            <mass value="1.0838"/>
+            <inertia ixx="0.008194" ixy="0.00015602" ixz="-3.434E-06" iyy="0.0011945" iyz="-0.00031298" izz="0.007915"/>
+        </inertial>
+        <collision>
+            <origin xyz="0 0 0" rpy="0 ${PI} 0"/>
+            <geometry>
+                <mesh filename="package://niryo_robot_description/meshes/ned2/stl/arm_link.stl"/>
+            </geometry>
+        </collision>
+    </link>
+    <link name="elbow_link">
+        <inertial>
+            <origin xyz="-0.019703 0.037336 -1.7431E-09" rpy="0 ${PI} 0"/>
+            <mass value="0.22126"/>
+            <inertia ixx="0.00011754" ixy="-1.2314E-05" ixz="-6.2064E-11" iyy="0.00020851" iyz="9.2393E-11"
+                     izz="0.00022753"/>
+        </inertial>
+        <collision>
+            <origin xyz="0 0 0" rpy="0 ${PI} 0"/>
+            <geometry>
+                <mesh filename="package://niryo_robot_description/meshes/ned2/stl/elbow_link.stl"/>
+            </geometry>
+        </collision>
+    </link>
+    <link name="forearm_link">
+        <inertial>
+            <origin xyz="-0.0049532 7.8351E-06 0.08106" rpy="0 0 0"/>
+            <mass value="0.35686"/>
+            <inertia ixx="0.0013664" ixy="-9.6367E-08" ixz="0.00013594" iyy="0.0014781" iyz="-1.4596E-07"
+                     izz="0.00023715"/>
+        </inertial>
         <collision>
             <origin xyz="0 0 0" rpy="0 0 0"/>
             <geometry>
-                <mesh filename="package://niryo_robot_description/meshes/ned2/stl/shoulder_link.stl"/>
-            </geometry>
-        </collision>
-    </link>
-    <link name="arm_link">
+                <mesh filename="package://niryo_robot_description/meshes/ned2/stl/forearm_link.stl"/>
+            </geometry>
+        </collision>
+    </link>
+    <!-- add collision for the motor of joint 5
+    <link name="joint5_motor">
+        <inertial>
+            <origin xyz="0 0 0.015" rpy="0 0 0"/>
+            <mass value="0.203543862275952"/>
+            <inertia ixx="0.0015" ixy="0.0" ixz="0.0" iyy="0.0015" iyz="0.0" izz="0.0015"/>
+        </inertial>
+        <collision>
+            <origin xyz="0 0 0.015" rpy="0 0 0"/>
+            <geometry>
+                <box size="0.047 0.0285 0.03"/>
+            </geometry>
+        </collision>
+    </link> -->
+    <link name="wrist_link">
+        <inertial>
+            <origin xyz="-0.019666 0.037312 0.0" rpy="0 0 0"/>
+            <mass value="0.22126"/>
+            <inertia ixx="0.0015" ixy="0.0" ixz="0.0" iyy="0.0015" iyz="0.0" izz="0.0015"/>
+        </inertial>
+        <collision>
+            <origin xyz="0 0 0"
+                    rpy="0 0 0"/>
+            <geometry>
+                <mesh filename="package://niryo_robot_description/meshes/ned2/stl/wrist_link.stl"/>
+            </geometry>
+        </collision>
+    </link>
+    <link name="hand_link">
+        <inertial>
+            <origin xyz="0 0 0.009" rpy="0 0 0"/>
+            <mass value="0.0070027"/>
+            <inertia ixx="0.0015" ixy="0.0" ixz="0.0" iyy="0.0015" iyz="0.0" izz="0.0015"/>
+        </inertial>
         <collision>
             <origin xyz="0 0 0" rpy="0 0 0"/>
             <geometry>
-                <mesh filename="package://niryo_robot_description/meshes/ned2/stl/arm_link.stl"/>
-            </geometry>
-        </collision>
-    </link>
-    <link name="elbow_link">
-        <collision>
-            <origin xyz="0 0 0" rpy="0 0 0"/>
-            <geometry>
-                <mesh filename="package://niryo_robot_description/meshes/ned2/stl/elbow_link.stl"/>
-            </geometry>
-        </collision>
-    </link>
-    <link name="forearm_link">
-        <collision>
-            <origin xyz="0 0 0" rpy="0 0 0"/>
-            <geometry>
-                <mesh filename="package://niryo_robot_description/meshes/ned2/stl/forearm_link.stl"/>
-            </geometry>
-        </collision>
-    </link>
-    <!-- add collision for the motor of joint 5 -->
-    <link name="joint5_motor">
-        <collision>
-            <origin xyz="0 0 0.015" rpy="0 0 0"/>
-            <geometry>
-                <box size="0.047 0.0285 0.03"/>
-            </geometry>
-        </collision>
-    </link>
-    <link name="wrist_link">
-        <collision>
-            <origin xyz="0 0 0" rpy="0 0 0"/>
-            <geometry>
-                <mesh filename="package://niryo_robot_description/meshes/ned2/stl/wrist_link.stl"/>
-            </geometry>
-        </collision>
-    </link>
-    <link name="hand_link">
-        <collision>
-            <origin xyz="0 0 0"  rpy="0 0 0"/>
-            <geometry>
                 <mesh filename="package://niryo_robot_description/meshes/ned2/stl/hand_link.stl"/>
             </geometry>
@@ -71,6 +130,4 @@
     </link>
     <link name="tool_link">
-    </link>
-    <link name="led_ring_link">
     </link>
     <!-- Joints -->
@@ -81,25 +138,25 @@
     </joint>
     <joint name="joint_1" type="revolute">
-        <origin xyz="0 3.7961E-05 0.1013" rpy="0 0 0"/>
+        <origin xyz="0 0 0.1013" rpy="0 0 ${-PI/2}"/>
         <parent link="base_link"/>
         <child link="shoulder_link"/>
         <axis xyz="0 0 1"/>
-        <limit effort="10.0" velocity="2.2" lower="${(limit_low_shoulder_rotation + safety_pos_margin) * deg_to_rad}"
+        <limit effort="10.0" velocity="10.0" lower="${(limit_low_shoulder_rotation + safety_pos_margin) * deg_to_rad}"
                upper="${(limit_up_shoulder_rotation - safety_pos_margin) * deg_to_rad}"/>
     </joint>
     <joint name="joint_2" type="revolute">
-        <origin xyz="0 0 0.065" rpy="${PI/2} ${-PI/2} 0"/>
+        <origin xyz="0 0 0.065" rpy="${PI/2} 0 ${PI/2}"/>
         <parent link="shoulder_link"/>
         <child link="arm_link"/>
         <axis xyz="0 0 1"/>
-        <limit effort="10.0" velocity="2.2" lower="${(limit_low_arm_rotation + safety_pos_margin) * deg_to_rad}"
+        <limit effort="10.0" velocity="8.0" lower="${(limit_low_arm_rotation + safety_pos_margin) * deg_to_rad}"
                upper="${(limit_up_arm_rotation - safety_pos_margin) * deg_to_rad}"/>
     </joint>
     <joint name="joint_3" type="revolute">
-        <origin xyz="0.221 -0.012 0" rpy="0 0 ${-PI/2}"/>
+        <origin xyz="0.012 0.221 0" rpy="0 0 0"/>
         <parent link="arm_link"/>
         <child link="elbow_link"/>
         <axis xyz="0 0 1"/>
-        <limit effort="7.0" velocity="2.0" lower="${(limit_low_elbow_rotation + safety_pos_margin) * deg_to_rad}"
+        <limit effort="7.0" velocity="8.0" lower="${(limit_low_elbow_rotation + safety_pos_margin) * deg_to_rad}"
                upper="${(limit_up_elbow_rotation - safety_pos_margin) * deg_to_rad}"/>
     </joint>
@@ -133,13 +190,14 @@
         <origin xyz="0 0 ${distance_hand_tool}" rpy="${-PI/2} ${-PI/2} 0"/>
     </joint>
+    <!--
     <joint name="joint_test" type="fixed">
         <origin xyz="-0.03 0 0.158" rpy="0 -${PI/2} 0"/>
         <parent link="forearm_link"/>
         <child link="joint5_motor"/>
-    </joint>
+    </joint> -->
     <joint name="joint_led_ring" type="fixed">
         <parent link="world"/>
         <child link="led_ring_link"/>
-        <origin xyz="0 0 0.0923" rpy="0 0 ${PI/2}"/>
+        <origin xyz="0 0 0.0923" rpy="0 0 0"/>
     </joint>
 </robot>
