Commit message: edit version number in various files

File: niryo_robot_description/urdf/ned/niryo_ned_camera.urdf.xacro (robot description, xacro)
@@ -21,5 +21,7 @@
                 <box size="${cameraWidth} ${cameraHeight} ${cameraHeight}"/>
             </geometry>
-            <material name="DarkGrey"/>
+            <material name="Grey">
+               <color rgba="0.7 0.7 0.7 1.0"/>
+            </material>
         </visual>
     </link>

File: niryo_robot_description/urdf/ned2/niryo_ned2_camera.urdf.xacro (robot description, xacro)
@@ -21,6 +21,15 @@
                 <box size="${cameraWidth} ${cameraHeight} ${cameraHeight}"/>
             </geometry>
-            <material name="DarkGrey"/>
+            <material name="Grey">
+               <color rgba="0.7 0.7 0.7 1.0"/>
+            </material>
         </visual>
+        <collision>
+            <origin xyz="0 0 0"
+                    rpy="0 0 0"/>
+            <geometry>
+                <box size="${cameraWidth} ${cameraHeight} ${cameraHeight}"/>
+            </geometry>
+        </collision>
     </link>
     <!-- Add gazebo settings to make the link an camera ! -->

File: niryo_robot_description/urdf/one/niryo_one_camera.urdf.xacro (robot description, xacro)
@@ -27,5 +27,7 @@
                 <box size="${cameraWidth} ${cameraWidth} ${cameraHeight}"/>
             </geometry>
-            <material name="DarkGrey"/>
+            <material name="Grey">
+               <color rgba="0.7 0.7 0.7 1.0"/>
+            </material>
         </visual>
         <inertial>
