Commit message: fix xacro collision for kinetic

File: niryo_robot_description/urdf/one/niryo_one.urdf.xacro (robot description, xacro)
@@ -139,4 +139,13 @@
     <link name="tool_link">
     </link>
+    <!-- add collision for the motor of joint 5 -->
+    <link name="joint5_motor">
+        <collision>
+            <origin xyz="-0.045 0.0 0.1765" rpy="0 0 0"/>
+            <geometry>
+                <box size="0.0435 0.0285 0.0465"/>
+            </geometry>
+        </collision>
+    </link>
     <!--Joints -->
     <joint name="joint_world" type="fixed">
@@ -179,21 +188,4 @@
         <dynamics damping="0.1" friction="0.0"/>
     </joint>
-      <!-- add collision for the motor of joint 5 -->
-    <link name="joint5_motor">
-        <inertial>
-            <origin xyz="-0.00811345462189901 -0.000135618649565461 0.107402242790047" rpy="0 0 0"/>
-            <mass value="0.203543862275952"/>
-            <inertia ixx="0.0015" ixy="0.0" ixz="0.0" iyy="0.0015" iyz="0.0" izz="0.0015"/>
-        </inertial>
-        <collision>
-            <origin xyz="-0.045 0.0 0.1765" rpy="0 0 0"/>
-            <geometry> <box size="0.0435 0.0285 0.0465"/> </geometry>
-        </collision>
-    </link>
-    <joint name="joint_test" type="fixed">
-        <origin xyz="0 0 0" rpy="0 0 0"/>
-        <parent link="forearm_link"/>
-        <child link="joint5_motor"/>
-    </joint>
     <joint name="joint_5" type="revolute">
         <parent link="forearm_link"/>
@@ -217,3 +209,9 @@
         <origin xyz="0 0 ${distance_hand_tool}" rpy="${-PI/2} ${-PI/2} 0"/>
     </joint>
+    <!-- add collision for the motor of joint 5 -->
+    <joint name="joint_test" type="fixed">
+        <origin xyz="0 0 0" rpy="0 0 0"/>
+        <parent link="forearm_link"/>
+        <child link="joint5_motor"/>
+    </joint>
 </robot>

File: niryo_robot_description/urdf/one/niryo_one_param.urdf.xacro (robot description, xacro)
@@ -13,5 +13,4 @@
     <xacro:property name="distance_wrist_hand_y" value="-0.0055" />
     <xacro:property name="distance_hand_tool" value="0.0073" />
-	<xacro:property name="PI" value="3.14159265359" />
     <xacro:property name="limit_low_shoulder_rotation" value="-3.05433" />
     <xacro:property name="limit_up_shoulder_rotation" value="3.05433" />

File: niryo_robot_description/urdf/one/without_mesh_niryo_one.urdf.xacro (robot description, xacro)
@@ -19,20 +19,14 @@
 	<!-- Links -->
     <link name="world"/>
-    <link name="base_link">
-	</link>
-    <link name="shoulder_link">
-	</link>
-    <link name="arm_link">
-	</link>
-    <link name="elbow_link">
-	</link>
-    <link name="forearm_link">
-	</link>
-    <link name="wrist_link">
-	</link>
-    <link name="hand_link">
-	</link>
-    <link name="tool_link">
-	</link>
+    <link name="base_link"/>
+    <link name="shoulder_link"/>
+    <link name="arm_link"/>
+    <link name="elbow_link"/>
+    <link name="forearm_link"/>
+    <link name="wrist_link"/>
+    <link name="hand_link"/>
+    <link name="tool_link"/>
+    <!-- add collision for the motor of joint 5 -->
+    <link name="joint5_motor"/>
 	<!--Joints -->
     <joint name="joint_world" type="fixed">
@@ -69,16 +63,4 @@
 		<axis xyz="0 0 1" />
 	</joint>
-	<!-- add collision for the motor of joint 5 -->
-    <link name="joint5_motor">
-        <collision>
-            <origin xyz="-0.045 0.0 0.1765" rpy="0 0 0"/>
-            <geometry> <box size="0.0435 0.0285 0.0465"/> </geometry>
-        </collision>
-    </link>
-    <joint name="joint_test"  type="fixed">
-        <origin xyz="0 0 0" rpy="0 0 0"/>
-        <parent link="forearm_link"/>
-        <child link="joint5_motor"/>
-    </joint>
 	<joint name="joint_5" type="revolute">
         <parent link="forearm_link" />
@@ -100,3 +82,9 @@
         <origin xyz="0 0 ${distance_hand_tool}" rpy="${-PI/2} ${-PI/2} 0" />
 	</joint>
+	<!-- add collision for the motor of joint 5 -->
+    <joint name="joint5_motor_joint" type="fixed">
+        <parent link="forearm_link" />
+        <child link="joint5_motor" />
+        <origin xyz="0 0 0" rpy="0 0 0" />
+	</joint>
 </robot>
