Commit message: small correction on ROS_WARN %lu not valid
correction for fake moveit with niryo one

small corrections on launch files in niryo_robot_bringup

correction on urdf for niryo one incorrect

File: niryo_robot_description/urdf/fake/niryo.transmission.xacro (robot description, xacro)
@@ -1,3 +1,3 @@
-<robot xmlns:xacro="http://ros.org/wiki/xacro" name="niryo_ned">
+<robot xmlns:xacro="http://ros.org/wiki/xacro">
   <!-- Transmission macro -->
   <xacro:macro name="SimpleTransmissionPosition" params="joint n">

File: niryo_robot_description/urdf/fake/niryo.urdf.xacro (robot description, xacro)
@@ -1,5 +1,5 @@
-<robot xmlns:xacro="http://www.ros.org/wiki/xacro" name="niryo_ned_2">
+<robot xmlns:xacro="http://www.ros.org/wiki/xacro" name="niryo_ned">
     <!-- Import Properties -->
-    <xacro:include filename="$(find niryo_robot_description)/urdf/ned2/niryo_param.urdf.xacro"/>
+    <xacro:include filename="$(find niryo_robot_description)/urdf/ned/niryo_param.urdf.xacro"/>
     <!-- Links -->
     <link name="world"/>
@@ -20,12 +20,12 @@
                     rpy="0 0 0"/>
             <geometry>
-                <mesh filename="package://niryo_robot_description/meshes/ned2/collada/base_link.dae"/>
-            </geometry>
-        </visual>
-        <collision>
-            <origin xyz="0 0 0"
-                    rpy="0 0 0"/>
-            <geometry>
-                <mesh filename="package://niryo_robot_description/meshes/ned2/stl/base_link.stl"/>
+                <mesh filename="package://niryo_robot_description/meshes/ned/collada/base_link.dae"/>
+            </geometry>
+        </visual>
+        <collision>
+            <origin xyz="0 0 0"
+                    rpy="0 0 0"/>
+            <geometry>
+                <mesh filename="package://niryo_robot_description/meshes/ned/stl/base_link.stl"/>
             </geometry>
         </collision>
@@ -52,12 +52,12 @@
                     rpy="0 0 0"/>
             <geometry>
-                <mesh filename="package://niryo_robot_description/meshes/ned2/collada/shoulder_link.dae"/>
-            </geometry>
-        </visual>
-        <collision>
-            <origin xyz="0 0 0"
-                    rpy="0 0 0"/>
-            <geometry>
-                <mesh filename="package://niryo_robot_description/meshes/ned2/stl/shoulder_link.stl"/>
+                <mesh filename="package://niryo_robot_description/meshes/ned/collada/shoulder_link.dae"/>
+            </geometry>
+        </visual>
+        <collision>
+            <origin xyz="0 0 0"
+                    rpy="0 0 0"/>
+            <geometry>
+                <mesh filename="package://niryo_robot_description/meshes/ned/stl/shoulder_link.stl"/>
             </geometry>
         </collision>
@@ -84,12 +84,12 @@
                     rpy="0 0 0"/>
             <geometry>
-                <mesh filename="package://niryo_robot_description/meshes/ned2/collada/arm_link.dae"/>
-            </geometry>
-        </visual>
-        <collision>
-            <origin xyz="0 0 0"
-                    rpy="0 0 0"/>
-            <geometry>
-                <mesh filename="package://niryo_robot_description/meshes/ned2/stl/arm_link.stl"/>
+                <mesh filename="package://niryo_robot_description/meshes/ned/collada/arm_link.dae"/>
+            </geometry>
+        </visual>
+        <collision>
+            <origin xyz="0 0 0"
+                    rpy="0 0 0"/>
+            <geometry>
+                <mesh filename="package://niryo_robot_description/meshes/ned/stl/arm_link.stl"/>
             </geometry>
         </collision>
@@ -116,12 +116,12 @@
                     rpy="0 0 0"/>
             <geometry>
-                <mesh filename="package://niryo_robot_description/meshes/ned2/collada/elbow_link.dae"/>
-            </geometry>
-        </visual>
-        <collision>
-            <origin xyz="0 0 0"
-                    rpy="0 0 0"/>
-            <geometry>
-                <mesh filename="package://niryo_robot_description/meshes/ned2/stl/elbow_link.stl"/>
+                <mesh filename="package://niryo_robot_description/meshes/ned/collada/elbow_link.dae"/>
+            </geometry>
+        </visual>
+        <collision>
+            <origin xyz="0 0 0"
+                    rpy="0 0 0"/>
+            <geometry>
+                <mesh filename="package://niryo_robot_description/meshes/ned/stl/elbow_link.stl"/>
             </geometry>
         </collision>
@@ -148,12 +148,12 @@
                     rpy="0 0 0"/>
             <geometry>
-                <mesh filename="package://niryo_robot_description/meshes/ned2/collada/forearm_link.dae"/>
-            </geometry>
-        </visual>
-        <collision>
-            <origin xyz="0 0 0"
-                    rpy="0 0 0"/>
-            <geometry>
-                <mesh filename="package://niryo_robot_description/meshes/ned2/stl/forearm_link.stl"/>
+                <mesh filename="package://niryo_robot_description/meshes/ned/collada/forearm_link.dae"/>
+            </geometry>
+        </visual>
+        <collision>
+            <origin xyz="0 0 0"
+                    rpy="0 0 0"/>
+            <geometry>
+                <mesh filename="package://niryo_robot_description/meshes/ned/stl/forearm_link.stl"/>
             </geometry>
         </collision>
@@ -204,12 +204,12 @@
                     rpy="0 0 0"/>
             <geometry>
-                <mesh filename="package://niryo_robot_description/meshes/ned2/collada/wrist_link.dae"/>
-            </geometry>
-        </visual>
-        <collision>
-            <origin xyz="0 0 0"
-                    rpy="0 0 0"/>
-            <geometry>
-                <mesh filename="package://niryo_robot_description/meshes/ned2/stl/wrist_link.stl"/>
+                <mesh filename="package://niryo_robot_description/meshes/ned/collada/wrist_link.dae"/>
+            </geometry>
+        </visual>
+        <collision>
+            <origin xyz="0 0 0"
+                    rpy="0 0 0"/>
+            <geometry>
+                <mesh filename="package://niryo_robot_description/meshes/ned/stl/wrist_link.stl"/>
             </geometry>
         </collision>
@@ -236,12 +236,12 @@
                     rpy="0 0 0"/>
             <geometry>
-                <mesh filename="package://niryo_robot_description/meshes/ned2/collada/hand_link.dae"/>
-            </geometry>
-        </visual>
-        <collision>
-            <origin xyz="0 0 0"
-                    rpy="0 0 0"/>
-            <geometry>
-                <mesh filename="package://niryo_robot_description/meshes/ned2/stl/hand_link.stl"/>
+                <mesh filename="package://niryo_robot_description/meshes/ned/collada/hand_link.dae"/>
+            </geometry>
+        </visual>
+        <collision>
+            <origin xyz="0 0 0"
+                    rpy="0 0 0"/>
+            <geometry>
+                <mesh filename="package://niryo_robot_description/meshes/ned/stl/hand_link.stl"/>
             </geometry>
         </collision>

File: niryo_robot_description/urdf/fake/niryo_camera.urdf.xacro (robot description, xacro)
@@ -1,5 +1,5 @@
-<robot xmlns:xacro="http://www.ros.org/wiki/xacro" name="niryo_ned_2">
+<robot xmlns:xacro="http://www.ros.org/wiki/xacro" name="niryo_ned">
     <!-- Including base robot -->
-    <xacro:include filename="$(find niryo_robot_description)/urdf/ned2/niryo_gazebo.urdf.xacro"/>
+    <xacro:include filename="$(find niryo_robot_description)/urdf/ned/niryo_gazebo.urdf.xacro"/>
     <!-- Properties -->
     <xacro:property name="cameraWidth" value="0.01"/>

File: niryo_robot_description/urdf/fake/niryo_gazebo.urdf.xacro (robot description, xacro)
@@ -1,3 +1,3 @@
-<robot xmlns:xacro="http://www.ros.org/wiki/xacro" name="niryo_ned_2">
+<robot xmlns:xacro="http://www.ros.org/wiki/xacro" name="niryo_ned">
     <!-- Enable Gazebo control-->
     <gazebo>
@@ -7,6 +7,6 @@
     </gazebo>
     <!-- Import Robot -->
-    <xacro:include filename="$(find niryo_robot_description)/urdf/ned2/niryo.urdf.xacro"/>
+    <xacro:include filename="$(find niryo_robot_description)/urdf/ned/niryo.urdf.xacro"/>
     <!-- Import Transmission -->
-    <xacro:include filename="$(find niryo_robot_description)/urdf/ned2/niryo.transmission.xacro"/>
+    <xacro:include filename="$(find niryo_robot_description)/urdf/ned/niryo.transmission.xacro"/>
 </robot>

File: niryo_robot_description/urdf/fake/niryo_gripper1_n_camera.urdf.xacro (robot description, xacro)
@@ -1,3 +1,3 @@
-<robot xmlns:xacro="http://www.ros.org/wiki/xacro" name="niryo_ned_2">
+<robot xmlns:xacro="http://www.ros.org/wiki/xacro" name="niryo_ned">
     <xacro:include filename="$(find niryo_robot_description)/urdf/ned/niryo_camera.urdf.xacro"/>
     <!-- gazebo joint state publisher for all joints. Necessary to control mors -->

File: niryo_robot_description/urdf/fake/niryo_param.urdf.xacro (robot description, xacro)
@@ -1,3 +1,3 @@
-<robot xmlns:xacro="http://www.ros.org/wiki/xacro" name="niryo_ned_2">
+<robot xmlns:xacro="http://www.ros.org/wiki/xacro" name="niryo_ned">
     <xacro:property name="PI" value="3.14159265359"/>
     <xacro:property name="deg_to_rad" value="${PI/180}"/>
@@ -12,6 +12,6 @@
     <xacro:property name="limit_low_forearm_rotation" value="-120.0"/>
     <xacro:property name="limit_up_forearm_rotation" value="120.0"/>
-    <xacro:property name="limit_low_wrist_rotation" value="-100.0"/>
-    <xacro:property name="limit_up_wrist_rotation" value="55.0"/>
+    <xacro:property name="limit_low_wrist_rotation" value="-120.0"/>
+    <xacro:property name="limit_up_wrist_rotation" value="60.0"/>
     <xacro:property name="limit_low_hand_rotation" value="-145.0"/>
     <xacro:property name="limit_up_hand_rotation" value="145.0"/>

File: niryo_robot_description/urdf/fake/without_mesh_niryo.urdf.xacro (robot description, xacro)
@@ -1,5 +1,5 @@
-<robot xmlns:xacro="http://www.ros.org/wiki/xacro" name="niryo_ned_2">
+<robot xmlns:xacro="http://www.ros.org/wiki/xacro" name="niryo_ned">
     <!-- Import Properties -->
-    <xacro:include filename="$(find niryo_robot_description)/urdf/ned2/niryo_param.urdf.xacro"/>
+    <xacro:include filename="$(find niryo_robot_description)/urdf/ned/niryo_param.urdf.xacro"/>
     <!-- Links -->
     <link name="world"/>
@@ -14,5 +14,5 @@
                     rpy="0 0 0"/>
             <geometry>
-                <mesh filename="package://niryo_robot_description/meshes/ned2/stl/base_link.stl"/>
+                <mesh filename="package://niryo_robot_description/meshes/ned/stl/base_link.stl"/>
             </geometry>
         </collision>
@@ -33,5 +33,5 @@
                     rpy="0 0 0"/>
             <geometry>
-                <mesh filename="package://niryo_robot_description/meshes/ned2/stl/shoulder_link.stl"/>
+                <mesh filename="package://niryo_robot_description/meshes/ned/stl/shoulder_link.stl"/>
             </geometry>
         </collision>
@@ -52,5 +52,5 @@
                     rpy="0 0 0"/>
             <geometry>
-                <mesh filename="package://niryo_robot_description/meshes/ned2/stl/arm_link.stl"/>
+                <mesh filename="package://niryo_robot_description/meshes/ned/stl/arm_link.stl"/>
             </geometry>
         </collision>
@@ -71,5 +71,5 @@
                     rpy="0 0 0"/>
             <geometry>
-                <mesh filename="package://niryo_robot_description/meshes/ned2/stl/elbow_link.stl"/>
+                <mesh filename="package://niryo_robot_description/meshes/ned/stl/elbow_link.stl"/>
             </geometry>
         </collision>
@@ -90,5 +90,5 @@
                     rpy="0 0 0"/>
             <geometry>
-                <mesh filename="package://niryo_robot_description/meshes/ned2/stl/forearm_link.stl"/>
+                <mesh filename="package://niryo_robot_description/meshes/ned/stl/forearm_link.stl"/>
             </geometry>
         </collision>
@@ -126,5 +126,5 @@
                     rpy="0 0 0"/>
             <geometry>
-                <mesh filename="package://niryo_robot_description/meshes/ned2/stl/wrist_link.stl"/>
+                <mesh filename="package://niryo_robot_description/meshes/ned/stl/wrist_link.stl"/>
             </geometry>
         </collision>
@@ -145,5 +145,5 @@
                     rpy="0 0 0"/>
             <geometry>
-                <mesh filename="package://niryo_robot_description/meshes/ned2/stl/hand_link.stl"/>
+                <mesh filename="package://niryo_robot_description/meshes/ned/stl/hand_link.stl"/>
             </geometry>
         </collision>

File: niryo_robot_description/urdf/ned2/niryo.transmission.xacro (robot description, xacro)
@@ -1,3 +1,3 @@
-<robot xmlns:xacro="http://ros.org/wiki/xacro">
+<robot xmlns:xacro="http://ros.org/wiki/xacro"  name="niryo_ned_2">
   <!-- Transmission macro -->
   <xacro:macro name="SimpleTransmissionPosition" params="joint n">

File: niryo_robot_description/urdf/one/niryo.transmission.xacro (robot description, xacro)
@@ -1,4 +1,4 @@
 <?xml version="1.0"?>
-<robot xmlns:xacro="http://ros.org/wiki/xacro">
+<robot xmlns:xacro="http://ros.org/wiki/xacro" name="niryo_one">
   <!-- Transmission macro -->
   <xacro:macro name="SimpleTransmissionPosition" params="joint n">

File: niryo_robot_description/urdf/one/niryo_gazebo.urdf.xacro (robot description, xacro)
@@ -5,5 +5,4 @@
         <plugin name="gazebo_ros_control" filename="libgazebo_ros_control.so">
             <robotSimType>gazebo_ros_control/DefaultRobotHWSim</robotSimType>
-<!--            <robotNamespace>/niryo_one</robotNamespace>-->
         </plugin>
     </gazebo>

File: niryo_robot_description/urdf/one/niryo_param.urdf.xacro (robot description, xacro)
@@ -1,3 +1,3 @@
-<robot xmlns:xacro="http://www.ros.org/wiki/xacro" name="niryo_ned">
+<robot xmlns:xacro="http://www.ros.org/wiki/xacro" name="niryo_one">
     <xacro:property name="PI" value="3.14159265359"/>
     <xacro:property name="deg_to_rad" value="${PI/180}"/>

File: niryo_robot_description/urdf/one/without_mesh_niryo.urdf.xacro (robot description, xacro)
@@ -1,5 +1,5 @@
 <?xml version="1.0"?>
 <!--
-    without_mesh_niryo_one.urdf.xacro
+    without_mesh_niryo.urdf.xacro
     Copyright (C) 2017 Niryo
     All rights reserved.
