Commit message: correction in progress for joints controller not loaded correctly

File: niryo_robot_description/urdf/fake/niryo.urdf.xacro (robot description, xacro)
@@ -21,12 +21,12 @@
                     rpy="0 0 0"/>
             <geometry>
-                <mesh filename="package://niryo_robot_description/meshes/ned/collada/base_link.dae"/>
-            </geometry>
-        </visual>
-        <collision>
-            <origin xyz="0 0 0"
-                    rpy="0 0 0"/>
-            <geometry>
-                <mesh filename="package://niryo_robot_description/meshes/ned/stl/base_link.stl"/>
+                <mesh filename="package://niryo_robot_description/meshes/fake/collada/base_link.dae"/>
+            </geometry>
+        </visual>
+        <collision>
+            <origin xyz="0 0 0"
+                    rpy="0 0 0"/>
+            <geometry>
+                <mesh filename="package://niryo_robot_description/meshes/fake/stl/base_link.stl"/>
             </geometry>
         </collision>
@@ -53,12 +53,12 @@
                     rpy="0 0 0"/>
             <geometry>
-                <mesh filename="package://niryo_robot_description/meshes/ned/collada/shoulder_link.dae"/>
-            </geometry>
-        </visual>
-        <collision>
-            <origin xyz="0 0 0"
-                    rpy="0 0 0"/>
-            <geometry>
-                <mesh filename="package://niryo_robot_description/meshes/ned/stl/shoulder_link.stl"/>
+                <mesh filename="package://niryo_robot_description/meshes/fake/collada/shoulder_link.dae"/>
+            </geometry>
+        </visual>
+        <collision>
+            <origin xyz="0 0 0"
+                    rpy="0 0 0"/>
+            <geometry>
+                <mesh filename="package://niryo_robot_description/meshes/fake/stl/shoulder_link.stl"/>
             </geometry>
         </collision>
@@ -85,12 +85,12 @@
                     rpy="0 0 0"/>
             <geometry>
-                <mesh filename="package://niryo_robot_description/meshes/ned/collada/arm_link.dae"/>
-            </geometry>
-        </visual>
-        <collision>
-            <origin xyz="0 0 0"
-                    rpy="0 0 0"/>
-            <geometry>
-                <mesh filename="package://niryo_robot_description/meshes/ned/stl/arm_link.stl"/>
+                <mesh filename="package://niryo_robot_description/meshes/fake/collada/arm_link.dae"/>
+            </geometry>
+        </visual>
+        <collision>
+            <origin xyz="0 0 0"
+                    rpy="0 0 0"/>
+            <geometry>
+                <mesh filename="package://niryo_robot_description/meshes/fake/stl/arm_link.stl"/>
             </geometry>
         </collision>
@@ -117,12 +117,12 @@
                     rpy="0 0 0"/>
             <geometry>
-                <mesh filename="package://niryo_robot_description/meshes/ned/collada/elbow_link.dae"/>
-            </geometry>
-        </visual>
-        <collision>
-            <origin xyz="0 0 0"
-                    rpy="0 0 0"/>
-            <geometry>
-                <mesh filename="package://niryo_robot_description/meshes/ned/stl/elbow_link.stl"/>
+                <mesh filename="package://niryo_robot_description/meshes/fake/collada/elbow_link.dae"/>
+            </geometry>
+        </visual>
+        <collision>
+            <origin xyz="0 0 0"
+                    rpy="0 0 0"/>
+            <geometry>
+                <mesh filename="package://niryo_robot_description/meshes/fake/stl/elbow_link.stl"/>
             </geometry>
         </collision>
@@ -149,12 +149,12 @@
                     rpy="0 0 0"/>
             <geometry>
-                <mesh filename="package://niryo_robot_description/meshes/ned/collada/forearm_link.dae"/>
-            </geometry>
-        </visual>
-        <collision>
-            <origin xyz="0 0 0"
-                    rpy="0 0 0"/>
-            <geometry>
-                <mesh filename="package://niryo_robot_description/meshes/ned/stl/forearm_link.stl"/>
+                <mesh filename="package://niryo_robot_description/meshes/fake/collada/forearm_link.dae"/>
+            </geometry>
+        </visual>
+        <collision>
+            <origin xyz="0 0 0"
+                    rpy="0 0 0"/>
+            <geometry>
+                <mesh filename="package://niryo_robot_description/meshes/fake/stl/forearm_link.stl"/>
             </geometry>
         </collision>
@@ -205,12 +205,12 @@
                     rpy="0 0 0"/>
             <geometry>
-                <mesh filename="package://niryo_robot_description/meshes/ned/collada/wrist_link.dae"/>
-            </geometry>
-        </visual>
-        <collision>
-            <origin xyz="0 0 0"
-                    rpy="0 0 0"/>
-            <geometry>
-                <mesh filename="package://niryo_robot_description/meshes/ned/stl/wrist_link.stl"/>
+                <mesh filename="package://niryo_robot_description/meshes/fake/collada/wrist_link.dae"/>
+            </geometry>
+        </visual>
+        <collision>
+            <origin xyz="0 0 0"
+                    rpy="0 0 0"/>
+            <geometry>
+                <mesh filename="package://niryo_robot_description/meshes/fake/stl/wrist_link.stl"/>
             </geometry>
         </collision>
@@ -237,12 +237,12 @@
                     rpy="0 0 0"/>
             <geometry>
-                <mesh filename="package://niryo_robot_description/meshes/ned/collada/hand_link.dae"/>
-            </geometry>
-        </visual>
-        <collision>
-            <origin xyz="0 0 0"
-                    rpy="0 0 0"/>
-            <geometry>
-                <mesh filename="package://niryo_robot_description/meshes/ned/stl/hand_link.stl"/>
+                <mesh filename="package://niryo_robot_description/meshes/fake/collada/hand_link.dae"/>
+            </geometry>
+        </visual>
+        <collision>
+            <origin xyz="0 0 0"
+                    rpy="0 0 0"/>
+            <geometry>
+                <mesh filename="package://niryo_robot_description/meshes/fake/stl/hand_link.stl"/>
             </geometry>
         </collision>

File: niryo_robot_description/urdf/fake/without_mesh_niryo.urdf.xacro (robot description, xacro)
@@ -15,5 +15,5 @@
                     rpy="0 0 0"/>
             <geometry>
-                <mesh filename="package://niryo_robot_description/meshes/ned/stl/base_link.stl"/>
+                <mesh filename="package://niryo_robot_description/meshes/fake/stl/base_link.stl"/>
             </geometry>
         </collision>
@@ -34,5 +34,5 @@
                     rpy="0 0 0"/>
             <geometry>
-                <mesh filename="package://niryo_robot_description/meshes/ned/stl/shoulder_link.stl"/>
+                <mesh filename="package://niryo_robot_description/meshes/fake/stl/shoulder_link.stl"/>
             </geometry>
         </collision>
@@ -53,5 +53,5 @@
                     rpy="0 0 0"/>
             <geometry>
-                <mesh filename="package://niryo_robot_description/meshes/ned/stl/arm_link.stl"/>
+                <mesh filename="package://niryo_robot_description/meshes/fake/stl/arm_link.stl"/>
             </geometry>
         </collision>
@@ -72,5 +72,5 @@
                     rpy="0 0 0"/>
             <geometry>
-                <mesh filename="package://niryo_robot_description/meshes/ned/stl/elbow_link.stl"/>
+                <mesh filename="package://niryo_robot_description/meshes/fake/stl/elbow_link.stl"/>
             </geometry>
         </collision>
@@ -91,5 +91,5 @@
                     rpy="0 0 0"/>
             <geometry>
-                <mesh filename="package://niryo_robot_description/meshes/ned/stl/forearm_link.stl"/>
+                <mesh filename="package://niryo_robot_description/meshes/fake/stl/forearm_link.stl"/>
             </geometry>
         </collision>
@@ -127,5 +127,5 @@
                     rpy="0 0 0"/>
             <geometry>
-                <mesh filename="package://niryo_robot_description/meshes/ned/stl/wrist_link.stl"/>
+                <mesh filename="package://niryo_robot_description/meshes/fake/stl/wrist_link.stl"/>
             </geometry>
         </collision>
@@ -146,5 +146,5 @@
                     rpy="0 0 0"/>
             <geometry>
-                <mesh filename="package://niryo_robot_description/meshes/ned/stl/hand_link.stl"/>
+                <mesh filename="package://niryo_robot_description/meshes/fake/stl/hand_link.stl"/>
             </geometry>
         </collision>
