Commit message: revert urdf names to niryo_$(hardware_version)

File: niryo_robot_description/urdf/ned2/niryo_ned2.urdf.xacro (robot description, xacro)
@@ -1,6 +1,6 @@
 <?xml version="1.0"?>
-<robot xmlns:xacro="http://www.ros.org/wiki/xacro" name="niryo_fake">
+<robot xmlns:xacro="http://www.ros.org/wiki/xacro" name="niryo_ned2">
     <!-- Import Properties -->
-    <xacro:include filename="$(find niryo_robot_description)/urdf/fake/niryo_param.urdf.xacro"/>
+    <xacro:include filename="$(find niryo_robot_description)/urdf/ned2/niryo_ned2_param.urdf.xacro"/>
     <!-- Links -->
     <link name="world"/>
@@ -21,12 +21,12 @@
                     rpy="0 0 0"/>
             <geometry>
-                <mesh filename="package://niryo_robot_description/meshes/fake/collada/base_link.dae"/>
-            </geometry>
-        </visual>
-        <collision>
-            <origin xyz="0 0 0"
-                    rpy="0 0 0"/>
-            <geometry>
-                <mesh filename="package://niryo_robot_description/meshes/fake/stl/base_link.stl"/>
+                <mesh filename="package://niryo_robot_description/meshes/ned2/collada/base_link.dae"/>
+            </geometry>
+        </visual>
+        <collision>
+            <origin xyz="0 0 0"
+                    rpy="0 0 0"/>
+            <geometry>
+                <mesh filename="package://niryo_robot_description/meshes/ned2/stl/base_link.stl"/>
             </geometry>
         </collision>
@@ -53,12 +53,12 @@
                     rpy="0 0 0"/>
             <geometry>
-                <mesh filename="package://niryo_robot_description/meshes/fake/collada/shoulder_link.dae"/>
-            </geometry>
-        </visual>
-        <collision>
-            <origin xyz="0 0 0"
-                    rpy="0 0 0"/>
-            <geometry>
-                <mesh filename="package://niryo_robot_description/meshes/fake/stl/shoulder_link.stl"/>
+                <mesh filename="package://niryo_robot_description/meshes/ned2/collada/shoulder_link.dae"/>
+            </geometry>
+        </visual>
+        <collision>
+            <origin xyz="0 0 0"
+                    rpy="0 0 0"/>
+            <geometry>
+                <mesh filename="package://niryo_robot_description/meshes/ned2/stl/shoulder_link.stl"/>
             </geometry>
         </collision>
@@ -85,12 +85,12 @@
                     rpy="0 0 0"/>
             <geometry>
-                <mesh filename="package://niryo_robot_description/meshes/fake/collada/arm_link.dae"/>
-            </geometry>
-        </visual>
-        <collision>
-            <origin xyz="0 0 0"
-                    rpy="0 0 0"/>
-            <geometry>
-                <mesh filename="package://niryo_robot_description/meshes/fake/stl/arm_link.stl"/>
+                <mesh filename="package://niryo_robot_description/meshes/ned2/collada/arm_link.dae"/>
+            </geometry>
+        </visual>
+        <collision>
+            <origin xyz="0 0 0"
+                    rpy="0 0 0"/>
+            <geometry>
+                <mesh filename="package://niryo_robot_description/meshes/ned2/stl/arm_link.stl"/>
             </geometry>
         </collision>
@@ -117,12 +117,12 @@
                     rpy="0 0 0"/>
             <geometry>
-                <mesh filename="package://niryo_robot_description/meshes/fake/collada/elbow_link.dae"/>
-            </geometry>
-        </visual>
-        <collision>
-            <origin xyz="0 0 0"
-                    rpy="0 0 0"/>
-            <geometry>
-                <mesh filename="package://niryo_robot_description/meshes/fake/stl/elbow_link.stl"/>
+                <mesh filename="package://niryo_robot_description/meshes/ned2/collada/elbow_link.dae"/>
+            </geometry>
+        </visual>
+        <collision>
+            <origin xyz="0 0 0"
+                    rpy="0 0 0"/>
+            <geometry>
+                <mesh filename="package://niryo_robot_description/meshes/ned2/stl/elbow_link.stl"/>
             </geometry>
         </collision>
@@ -149,12 +149,12 @@
                     rpy="0 0 0"/>
             <geometry>
-                <mesh filename="package://niryo_robot_description/meshes/fake/collada/forearm_link.dae"/>
-            </geometry>
-        </visual>
-        <collision>
-            <origin xyz="0 0 0"
-                    rpy="0 0 0"/>
-            <geometry>
-                <mesh filename="package://niryo_robot_description/meshes/fake/stl/forearm_link.stl"/>
+                <mesh filename="package://niryo_robot_description/meshes/ned2/collada/forearm_link.dae"/>
+            </geometry>
+        </visual>
+        <collision>
+            <origin xyz="0 0 0"
+                    rpy="0 0 0"/>
+            <geometry>
+                <mesh filename="package://niryo_robot_description/meshes/ned2/stl/forearm_link.stl"/>
             </geometry>
         </collision>
@@ -205,12 +205,12 @@
                     rpy="0 0 0"/>
             <geometry>
-                <mesh filename="package://niryo_robot_description/meshes/fake/collada/wrist_link.dae"/>
-            </geometry>
-        </visual>
-        <collision>
-            <origin xyz="0 0 0"
-                    rpy="0 0 0"/>
-            <geometry>
-                <mesh filename="package://niryo_robot_description/meshes/fake/stl/wrist_link.stl"/>
+                <mesh filename="package://niryo_robot_description/meshes/ned2/collada/wrist_link.dae"/>
+            </geometry>
+        </visual>
+        <collision>
+            <origin xyz="0 0 0"
+                    rpy="0 0 0"/>
+            <geometry>
+                <mesh filename="package://niryo_robot_description/meshes/ned2/stl/wrist_link.stl"/>
             </geometry>
         </collision>
@@ -237,12 +237,12 @@
                     rpy="0 0 0"/>
             <geometry>
-                <mesh filename="package://niryo_robot_description/meshes/fake/collada/hand_link.dae"/>
-            </geometry>
-        </visual>
-        <collision>
-            <origin xyz="0 0 0"
-                    rpy="0 0 0"/>
-            <geometry>
-                <mesh filename="package://niryo_robot_description/meshes/fake/stl/hand_link.stl"/>
+                <mesh filename="package://niryo_robot_description/meshes/ned2/collada/hand_link.dae"/>
+            </geometry>
+        </visual>
+        <collision>
+            <origin xyz="0 0 0"
+                    rpy="0 0 0"/>
+            <geometry>
+                <mesh filename="package://niryo_robot_description/meshes/ned2/stl/hand_link.stl"/>
             </geometry>
         </collision>

File: niryo_robot_description/urdf/ned2/niryo_ned2_camera.urdf.xacro (robot description, xacro)
@@ -2,5 +2,5 @@
 <robot xmlns:xacro="http://www.ros.org/wiki/xacro" name="niryo_ned2">
     <!-- Including base robot -->
-    <xacro:include filename="$(find niryo_robot_description)/urdf/ned2/niryo_gazebo.urdf.xacro"/>
+    <xacro:include filename="$(find niryo_robot_description)/urdf/ned2/niryo_ned2_gazebo.urdf.xacro"/>
     <!-- Properties -->
     <xacro:property name="cameraWidth" value="0.01"/>

File: niryo_robot_description/urdf/ned2/niryo_ned2_gazebo.urdf.xacro (robot description, xacro)
@@ -1,4 +1,4 @@
 <?xml version="1.0"?>
-<robot xmlns:xacro="http://www.ros.org/wiki/xacro" name="niryo_fake">
+<robot xmlns:xacro="http://www.ros.org/wiki/xacro" name="niryo_ned2">
     <!-- Enable Gazebo control-->
     <gazebo>
@@ -8,6 +8,6 @@
     </gazebo>
     <!-- Import Robot -->
-    <xacro:include filename="$(find niryo_robot_description)/urdf/fake/niryo.urdf.xacro"/>
+    <xacro:include filename="$(find niryo_robot_description)/urdf/ned2/niryo_ned2.urdf.xacro"/>
     <!-- Import Transmission -->
-    <xacro:include filename="$(find niryo_robot_description)/urdf/fake/niryo.transmission.xacro"/>
+    <xacro:include filename="$(find niryo_robot_description)/urdf/ned2/niryo_ned2.transmission.xacro"/>
 </robot>

File: niryo_robot_description/urdf/ned2/niryo_ned2_gripper1_n_camera.urdf.xacro (robot description, xacro)
@@ -1,5 +1,5 @@
 <?xml version="1.0"?>
-<robot xmlns:xacro="http://www.ros.org/wiki/xacro" name="niryo_one">
-    <xacro:include filename="$(find niryo_robot_description)/urdf/one/niryo_camera.urdf.xacro"/>
+<robot xmlns:xacro="http://www.ros.org/wiki/xacro" name="niryo_ned2">
+    <xacro:include filename="$(find niryo_robot_description)/urdf/ned2/niryo_ned2_camera.urdf.xacro"/>
     <!-- gazebo joint state publisher for all joints. Necessary to control mors -->
     <gazebo>
@@ -17,5 +17,5 @@
         <child link="base_gripper_1"/>
         <origin
-                xyz="0 0 0"
+                xyz="0 0 0.005"
                 rpy="0 ${PI/2} ${PI/2}"/>
     </joint>
@@ -39,5 +39,5 @@
             <geometry>
                 <mesh
-                        filename="package://niryo_robot_description/meshes/gripper_1/base_gripper_1.STL"/>
+                        filename="package://niryo_robot_description/meshes/ned2/gripper_1/base_gripper_1.STL"/>
             </geometry>
         </visual>
@@ -47,5 +47,5 @@
             <geometry>
                 <mesh
-                        filename="package://niryo_robot_description/meshes/gripper_1/base_gripper_1.STL"/>
+                        filename="package://niryo_robot_description/meshes/ned2/gripper_1/base_gripper_1.STL"/>
             </geometry>
         </collision>
@@ -71,5 +71,5 @@
             <geometry>
                 <mesh
-                        filename="package://niryo_robot_description/meshes/gripper_1/mors_1.STL"/>
+                        filename="package://niryo_robot_description/meshes/ned2/gripper_1/mors_1.STL"/>
             </geometry>
             <material name="">
@@ -82,5 +82,5 @@
             <geometry>
                 <mesh
-                        filename="package://niryo_robot_description/meshes/gripper_1/mors_1.STL"/>
+                        filename="package://niryo_robot_description/meshes/ned2/gripper_1/mors_1.STL"/>
             </geometry>
         </collision>
@@ -119,5 +119,5 @@
             <geometry>
                 <mesh
-                        filename="package://niryo_robot_description/meshes/gripper_1/mors_2.STL"/>
+                        filename="package://niryo_robot_description/meshes/ned2/gripper_1/mors_2.STL"/>
             </geometry>
         </visual>
@@ -127,5 +127,5 @@
             <geometry>
                 <mesh
-                        filename="package://niryo_robot_description/meshes/gripper_1/mors_2.STL"/>
+                        filename="package://niryo_robot_description/meshes/ned2/gripper_1/mors_2.STL"/>
             </geometry>
         </collision>

File: niryo_robot_description/urdf/ned2/without_mesh_niryo_ned2.urdf.xacro (robot description, xacro)
@@ -2,5 +2,5 @@
 <robot xmlns:xacro="http://www.ros.org/wiki/xacro" name="niryo_ned2">
     <!-- Import Properties -->
-    <xacro:include filename="$(find niryo_robot_description)/urdf/ned2/niryo_param.urdf.xacro"/>
+    <xacro:include filename="$(find niryo_robot_description)/urdf/ned2/niryo_ned2_param.urdf.xacro"/>
     <!-- Links -->
     <link name="world"/>

File: niryo_robot_description/urdf/one/niryo_one.urdf.xacro (robot description, xacro)
@@ -2,5 +2,5 @@
 <robot xmlns:xacro="http://www.ros.org/wiki/xacro" name="niryo_one">
     <!-- Properties -->
-    <xacro:include filename="$(find niryo_robot_description)/urdf/one/niryo_param.urdf.xacro"/>
+    <xacro:include filename="$(find niryo_robot_description)/urdf/one/niryo_one_param.urdf.xacro"/>
     <!-- Links -->
     <link name="world"/>

File: niryo_robot_description/urdf/one/niryo_one_camera.urdf.xacro (robot description, xacro)
@@ -1,14 +1,14 @@
 <?xml version="1.0"?>
-<robot xmlns:xacro="http://www.ros.org/wiki/xacro" name="niryo_ned">
+<robot xmlns:xacro="http://www.ros.org/wiki/xacro" name="niryo_one">
     <!-- Including base robot -->
-    <xacro:include filename="$(find niryo_robot_description)/urdf/ned/niryo_gazebo.urdf.xacro"/>
+    <xacro:include filename="$(find niryo_robot_description)/urdf/one/niryo_one_gazebo.urdf.xacro"/>
     <!-- Properties -->
-    <xacro:property name="cameraWidth" value="0.01"/>
-    <xacro:property name="cameraHeight" value="0.037"/>
+    <xacro:property name="cameraWidth" value="0.03"/>
+    <xacro:property name="cameraHeight" value="0.02"/>
     <xacro:property name="cameraMass" value="0.05"/>
     <!-- Joint for camera -->
     <joint name="camera_joint" type="fixed">
         <axis xyz="0 0 1"/>
-        <origin xyz="0 ${cameraHeight/2 + 0.02} 0" rpy="-${PI/2} 0 0"/>
+        <origin xyz="0 0.025 0" rpy="-${PI/2} 0 0"/>
         <parent link="wrist_link"/>
         <child link="camera_link"/>
@@ -16,11 +16,22 @@
     <!-- Camera link -->
     <link name="camera_link">
+        <collision>
+            <origin xyz="0 0 0" rpy="0 0 0"/>
+            <geometry>
+                <box size="${cameraWidth} ${cameraWidth} ${cameraHeight}"/>
+            </geometry>
+        </collision>
         <visual>
             <origin xyz="0 0 0" rpy="0 0 0"/>
             <geometry>
-                <box size="${cameraWidth} ${cameraHeight} ${cameraHeight}"/>
+                <box size="${cameraWidth} ${cameraWidth} ${cameraHeight}"/>
             </geometry>
             <material name="DarkGrey"/>
         </visual>
+        <inertial>
+            <mass value="${cameraMass}"/>
+            <origin xyz="0 0 0" rpy="0 0 0"/>
+            <inertia ixx="5.4e-6" ixy="0" ixz="0" iyy="5.4e-6" iyz="0" izz="7.5e-6"/>
+        </inertial>
     </link>
     <!-- Add gazebo settings to make the link an camera ! -->

File: niryo_robot_description/urdf/one/niryo_one_gazebo.urdf.xacro (robot description, xacro)
@@ -8,6 +8,6 @@
     </gazebo>
     <!-- Import Robot -->
-    <xacro:include filename="$(find niryo_robot_description)/urdf/one/niryo.urdf.xacro"/>
+    <xacro:include filename="$(find niryo_robot_description)/urdf/one/niryo_one.urdf.xacro"/>
     <!-- Import Transmission -->
-    <xacro:include filename="$(find niryo_robot_description)/urdf/one/niryo.transmission.xacro"/>
+    <xacro:include filename="$(find niryo_robot_description)/urdf/one/niryo_one.transmission.xacro"/>
 </robot>

File: niryo_robot_description/urdf/one/niryo_one_gripper1_n_camera.urdf.xacro (robot description, xacro)
@@ -1,5 +1,5 @@
 <?xml version="1.0"?>
-<robot xmlns:xacro="http://www.ros.org/wiki/xacro" name="niryo_ned">
-    <xacro:include filename="$(find niryo_robot_description)/urdf/ned/niryo_camera.urdf.xacro"/>
+<robot xmlns:xacro="http://www.ros.org/wiki/xacro" name="niryo_one">
+    <xacro:include filename="$(find niryo_robot_description)/urdf/one/niryo_one_camera.urdf.xacro"/>
     <!-- gazebo joint state publisher for all joints. Necessary to control mors -->
     <gazebo>
@@ -17,5 +17,5 @@
         <child link="base_gripper_1"/>
         <origin
-                xyz="0 0 0.005"
+                xyz="0 0 0"
                 rpy="0 ${PI/2} ${PI/2}"/>
     </joint>
@@ -39,5 +39,5 @@
             <geometry>
                 <mesh
-                        filename="package://niryo_robot_description/meshes/gripper_1/base_gripper_1.STL"/>
+                        filename="package://niryo_robot_description/meshes/one/gripper_1/base_gripper_1.STL"/>
             </geometry>
         </visual>
@@ -47,5 +47,5 @@
             <geometry>
                 <mesh
-                        filename="package://niryo_robot_description/meshes/gripper_1/base_gripper_1.STL"/>
+                        filename="package://niryo_robot_description/meshes/one/gripper_1/base_gripper_1.STL"/>
             </geometry>
         </collision>
@@ -71,5 +71,5 @@
             <geometry>
                 <mesh
-                        filename="package://niryo_robot_description/meshes/gripper_1/mors_1.STL"/>
+                        filename="package://niryo_robot_description/meshes/one/gripper_1/mors_1.STL"/>
             </geometry>
             <material name="">
@@ -82,5 +82,5 @@
             <geometry>
                 <mesh
-                        filename="package://niryo_robot_description/meshes/gripper_1/mors_1.STL"/>
+                        filename="package://niryo_robot_description/meshes/one/gripper_1/mors_1.STL"/>
             </geometry>
         </collision>
@@ -119,5 +119,5 @@
             <geometry>
                 <mesh
-                        filename="package://niryo_robot_description/meshes/gripper_1/mors_2.STL"/>
+                        filename="package://niryo_robot_description/meshes/one/gripper_1/mors_2.STL"/>
             </geometry>
         </visual>
@@ -127,5 +127,5 @@
             <geometry>
                 <mesh
-                        filename="package://niryo_robot_description/meshes/gripper_1/mors_2.STL"/>
+                        filename="package://niryo_robot_description/meshes/one/gripper_1/mors_2.STL"/>
             </geometry>
         </collision>

File: niryo_robot_description/urdf/one/without_mesh_niryo_one.urdf.xacro (robot description, xacro)
@@ -1,6 +1,6 @@
 <?xml version="1.0"?>
 <!--
-    without_mesh_niryo.urdf.xacro
-    Copyright (C) 2017 Niryo
+    without_mesh_niryo_one.urdf.xacro
+    Copyright (C) 2020 Niryo
     All rights reserved.
     This program is free software: you can redistribute it and/or modify
@@ -16,5 +16,5 @@
 -->
 <robot xmlns:xacro="http://www.ros.org/wiki/xacro" name="niryo_one">
-    <xacro:include filename="$(find niryo_robot_description)/urdf/one/niryo_param.urdf.xacro"/>
+    <xacro:include filename="$(find niryo_robot_description)/urdf/one/niryo_one_param.urdf.xacro"/>
 	<!-- Links -->
     <link name="world"/>
