Commit message: fix gazebo simu

File: niryo_robot_description/urdf/ned2/niryo_ned2_camera.urdf.xacro (robot description, xacro)
@@ -10,5 +10,5 @@
     <joint name="camera_joint" type="fixed">
         <axis xyz="0 0 1"/>
-        <origin xyz="0 ${cameraHeight/2 + 0.02} 0" rpy="-${PI/2} 0 0"/>
+        <origin xyz="0 ${cameraHeight/2 + 0.02} 0" rpy="${PI/2} 0 0"/>
         <parent link="wrist_link"/>
         <child link="camera_link"/>

Commit message: fix: SN-541 Fix camera and gripper transforms in ned3pro and ned2 URDF for simulation

File: niryo_robot_description/urdf/ned2/niryo_ned2_camera.urdf.xacro (robot description, xacro)
@@ -10,5 +10,5 @@
     <joint name="camera_joint" type="fixed">
         <axis xyz="0 0 1"/>
-        <origin xyz="0 ${cameraHeight/2 + 0.02} 0" rpy="${PI/2} 0 ${deg_to_rad*10}"/>
+        <origin xyz="${cameraHeight/2 + 0.02} 0 0" rpy="0 0 ${-PI/2+deg_to_rad*10}"/>
         <parent link="wrist_link"/>
         <child link="camera_link"/>

File: niryo_robot_description/urdf/ned2/niryo_ned2_gripper1_n_camera.urdf.xacro (robot description, xacro)
@@ -17,6 +17,6 @@
         <child link="base_gripper_1"/>
         <origin
-                xyz="0.003 0 -0.007"
-                rpy="0 ${-PI/2} ${PI/2}"/>
+                xyz="-0.007 0 0.003"
+                rpy="${-PI/2} 0 0"/>
     </joint>
     <!-- Base Gripper -->

File: niryo_robot_description/urdf/ned3pro/niryo_ned3pro_camera.urdf.xacro (robot description, xacro)
@@ -10,5 +10,5 @@
     <joint name="camera_joint" type="fixed">
         <axis xyz="0 0 1"/>
-        <origin xyz="0 ${cameraHeight/2 + 0.02} 0" rpy="${PI/2} 0 ${deg_to_rad*10}"/>
+        <origin xyz="${cameraHeight/2 + 0.02} 0 0" rpy="0 0 ${-PI/2+0.174533}"/>
         <parent link="wrist_link"/>
         <child link="camera_link"/>

File: niryo_robot_description/urdf/ned3pro/niryo_ned3pro_gripper1_n_camera.urdf.xacro (robot description, xacro)
@@ -17,6 +17,6 @@
         <child link="base_gripper_1"/>
         <origin
-                xyz="0.003 0 -0.007"
-                rpy="0 ${-PI/2} ${PI/2}"/>
+                xyz="-0.007 0 0.003"
+                rpy="${-PI/2} 0 0"/>
     </joint>
     <!-- Base Gripper -->
