Commit message: add velocity in urdf

File: niryo_robot_description/urdf/ned2/niryo_ned2.urdf.xacro (robot description, xacro)
@@ -39,5 +39,5 @@
         <child link="shoulder_link"/>
         <axis xyz="0 0 1"/>
-        <limit effort="10.0" velocity="2.2" lower="${(limit_low_shoulder_rotation + safety_pos_margin) * deg_to_rad}"
+        <limit effort="10.0" velocity="10.0" lower="${(limit_low_shoulder_rotation + safety_pos_margin) * deg_to_rad}"
                upper="${(limit_up_shoulder_rotation - safety_pos_margin) * deg_to_rad}"/>
     </joint>
@@ -71,5 +71,5 @@
         <child link="arm_link"/>
         <axis xyz="0 0 1"/>
-        <limit effort="10.0" velocity="2.2" lower="${(limit_low_arm_rotation + safety_pos_margin) * deg_to_rad}"
+        <limit effort="10.0" velocity="8.0" lower="${(limit_low_arm_rotation + safety_pos_margin) * deg_to_rad}"
                upper="${(limit_up_arm_rotation - safety_pos_margin) * deg_to_rad}"/>
     </joint>
@@ -103,5 +103,5 @@
         <child link="elbow_link"/>
         <axis xyz="0 0 1"/>
-        <limit effort="7.0" velocity="2.0" lower="${(limit_low_elbow_rotation + safety_pos_margin) * deg_to_rad}"
+        <limit effort="7.0" velocity="8.0" lower="${(limit_low_elbow_rotation + safety_pos_margin) * deg_to_rad}"
                upper="${(limit_up_elbow_rotation - safety_pos_margin) * deg_to_rad}"/>
     </joint>

Commit message: Urdf ned2

File: niryo_robot_description/urdf/ned2/niryo_ned2.urdf.xacro (robot description, xacro)
@@ -5,4 +5,182 @@
     <!-- Links -->
     <link name="world"/>
+    <link name="base_link">
+        <inertial>
+            <origin xyz="-0.008924 0.0001357 0.052392" rpy="0 0 0"/>
+            <mass value="0.71142"/>
+            <inertia ixx="0.0017" ixy="0.0" ixz="0.0" iyy="0.0017" iyz="0.0" izz="0.0032"/>
+        </inertial>
+        <visual>
+            <origin xyz="0 0 0" rpy="0 0 0"/>
+            <geometry>
+                <mesh filename="package://niryo_robot_description/meshes/ned2/collada/base_link.dae"/>
+            </geometry>
+        </visual>
+        <collision>
+            <origin xyz="0 0 0" rpy="-${PI/2} 0 0"/>
+            <geometry>
+                <mesh filename="package://niryo_robot_description/meshes/ned2/stl/base_link.stl"/>
+            </geometry>
+        </collision>
+    </link>
+    <link name="led_ring_link">
+        <!--
+        <visual>
+            <origin xyz="0 0 0"
+                    rpy="0 0 0"/>
+            <geometry>
+                <cylinder length="0.0019" radius="0.0775"/>
+            </geometry>
+            <material
+                    name="">
+                <color
+                        rgba="1 1 1 0.25"/>
+            </material>
+        </visual> -->
+    </link>
+    <link name="shoulder_link">
+        <inertial>
+            <origin xyz="-0.031951 0.0080419 0.030675" rpy="0 0 0"/>
+            <mass value="0.35056"/>
+            <inertia ixx="0.00023875" ixy="2.3853E-08" ixz="2.0596E-06" iyy="0.00032638" iyz="-8.9319E-07"
+                     izz="0.00030089"/>
+        </inertial>
+        <visual>
+            <origin xyz="0 0 0" rpy="0 0 0"/>
+            <geometry>
+                <mesh filename="package://niryo_robot_description/meshes/ned2/collada/shoulder_link.dae"/>
+            </geometry>
+        </visual>
+        <collision>
+            <origin xyz="0 0 0" rpy="0 0 0"/>
+            <geometry>
+                <mesh filename="package://niryo_robot_description/meshes/ned2/stl/shoulder_link.stl"/>
+            </geometry>
+        </collision>
+    </link>
+    <link name="arm_link">
+        <inertial>
+            <origin xyz="0.116485160625991 -0.00141190194997476 -0.00338105503061108"
+                    rpy="0 0 0"/>
+            <mass value="0.513332159226246"/>
+            <inertia ixx="0.0015" ixy="0.0" ixz="0.0" iyy="0.0015" iyz="0.0" izz="0.0015"/>
+        </inertial>
+        <visual>
+            <origin xyz="0 0 0"
+                    rpy="0 0 0"/>
+            <geometry>
+                <mesh filename="package://niryo_robot_description/meshes/ned2/collada/arm_link.dae"/>
+            </geometry>
+        </visual>
+        <collision>
+            <origin xyz="0 0 0"
+                    rpy="0 0 0"/>
+            <geometry>
+                <mesh filename="package://niryo_robot_description/meshes/ned2/stl/arm_link.stl"/>
+            </geometry>
+        </collision>
+    </link>
+    <link name="elbow_link">
+        <inertial>
+            <origin
+                    xyz="0.0082004 0.023746 0.0053676" rpy="0 0 0"/>
+            <mass value="0.15494"/>
+            <inertia ixx="6.0879E-05" ixy="-1.2086E-05" ixz="-1.3026E-08" iyy="7.4479E-05" iyz="-4.6729E-08"
+                     izz="9.8727E-05"/>
+        </inertial>
+        <visual>
+            <origin xyz="0 0 0"
+                    rpy="0 0 0"/>
+            <geometry>
+                <mesh filename="package://niryo_robot_description/meshes/ned2/collada/elbow_link.dae"/>
+            </geometry>
+        </visual>
+        <collision>
+            <origin xyz="0 0 0"
+                    rpy="0 0 0"/>
+            <geometry>
+                <mesh filename="package://niryo_robot_description/meshes/ned2/stl/elbow_link.stl"/>
+            </geometry>
+        </collision>
+    </link>
+    <link name="forearm_link">
+        <inertial>
+            <origin xyz="-0.0094603 8.5954E-05 0.10662" rpy="0 0 0"/>
+            <mass value="0.16445"/>
+            <inertia ixx="0.00015109" ixy="-1.6205E-07" ixz="4.3654E-07" iyy="0.00014456" iyz="-3.9296E-07"
+                     izz="4.8807E-05"/>
+        </inertial>
+        <visual>
+            <origin xyz="0 0 0" rpy="0 0 0"/>
+            <geometry>
+                <mesh filename="package://niryo_robot_description/meshes/ned2/collada/forearm_link.dae"/>
+            </geometry>
+        </visual>
+        <collision>
+            <origin xyz="0 0 0" rpy="0 0 0"/>
+            <geometry>
+                <mesh filename="package://niryo_robot_description/meshes/ned2/stl/forearm_link.stl"/>
+            </geometry>
+        </collision>
+    </link>
+    <!-- add collision for the motor of joint 5 -->
+    <link name="joint5_motor">
+        <inertial>
+            <origin xyz="-0.00811345462189901 -0.000135618649565461 0.107402242790047"
+                    rpy="0 0 0"/>
+            <mass value="0.203543862275952"/>
+            <inertia ixx="0.0015" ixy="0.0" ixz="0.0" iyy="0.0015" iyz="0.0" izz="0.0015"/>
+        </inertial>
+        <collision>
+            <origin xyz="0 0 0.015" rpy="0 0 0"/>
+            <geometry>
+                <box size="0.047 0.0285 0.03"/>
+            </geometry>
+        </collision>
+    </link>
+    <link name="wrist_link">
+        <inertial>
+            <origin xyz="-0.020082 0.0015621 9.3782E-05" rpy="0 0 0"/>
+            <mass value="0.03067"/>
+            <inertia ixx="4.2466E-06" ixy="-2.9761E-07" ixz="-9.1198E-09" iyy="3.6068E-06" iyz="-3.5847E-08"
+                     izz="3.801E-06"/>
+        </inertial>
+        <visual>
+            <origin xyz="0 0 0"
+                    rpy="0 0 0"/>
+            <geometry>
+                <mesh filename="package://niryo_robot_description/meshes/ned2/collada/wrist_link.dae"/>
+            </geometry>
+        </visual>
+        <collision>
+            <origin xyz="0 0 0"
+                    rpy="0 0 0"/>
+            <geometry>
+                <mesh filename="package://niryo_robot_description/meshes/ned2/stl/wrist_link.stl"/>
+            </geometry>
+        </collision>
+    </link>
+    <link name="hand_link">
+        <inertial>
+            <origin xyz="0 0 0.009" rpy="0 0 0"/>
+            <mass value="0.0070027"/>
+            <inertia ixx="0.0015" ixy="0.0" ixz="0.0" iyy="0.0015" iyz="0.0" izz="0.0015"/>
+        </inertial>
+        <visual>
+            <origin xyz="0 0 0" rpy="0 0 0"/>
+            <geometry>
+                <mesh filename="package://niryo_robot_description/meshes/ned2/collada/hand_link.dae"/>
+            </geometry>
+        </visual>
+        <collision>
+            <origin xyz="0 0 0" rpy="0 0 0"/>
+            <geometry>
+                <mesh filename="package://niryo_robot_description/meshes/ned2/stl/hand_link.stl"/>
+            </geometry>
+        </collision>
+    </link>
+    <link name="tool_link">
+    </link>
+    <!-- Joints -->
     <joint name="joint_world" type="fixed">
         <parent link="world"/>
@@ -10,30 +188,11 @@
         <origin xyz="0 0 0" rpy="0 0 0"/>
     </joint>
-    <link name="base_link">
-        <inertial>
-            <origin xyz="-0.00240796011216664 -0.00591764669105095 0.0515774030380053"
-                    rpy="0 0 0"/>
-            <mass value="0.999243361008122"/>
-            <inertia ixx="0.002" ixy="0.0" ixz="0.0" iyy="0.002" iyz="0.0" izz="0.004"/>
-        </inertial>
-        <visual>
-            <origin xyz="0 0 0"
-                    rpy="0 0 0"/>
-            <geometry>
-                <mesh filename="package://niryo_robot_description/meshes/ned2/collada/base_link.dae"/>
-            </geometry>
-        </visual>
-        <collision>
-            <origin xyz="0 0 0"
-                    rpy="0 0 0"/>
-            <geometry>
-                <mesh filename="package://niryo_robot_description/meshes/ned2/stl/base_link.stl"/>
-            </geometry>
-        </collision>
-    </link>
-    <joint name="joint_1"
-           type="revolute">
-        <origin xyz="0 0 0.1065"
-                rpy="0 0 0"/>
+    <joint name="joit_led_ring" type="fixed">
+        <parent link="world"/>
+        <child link="led_ring_link"/>
+        <origin xyz="0 0 0.0923" rpy="0 0 0"/>
+    </joint>
+    <joint name="joint_1" type="revolute">
+        <origin xyz="0 3.7961E-05 0.1013" rpy="0 0 0"/>
         <parent link="base_link"/>
         <child link="shoulder_link"/>
@@ -42,30 +201,6 @@
                upper="${(limit_up_shoulder_rotation - safety_pos_margin) * deg_to_rad}"/>
     </joint>
-    <link name="shoulder_link">
-        <inertial>
-            <origin xyz="-0.0307310771918448 0.00581074732334248 0.0302277607274943"
-                    rpy="0 0 0"/>
-            <mass value="0.474558968160783"/>
-            <inertia ixx="0.0015" ixy="0.0" ixz="0.0" iyy="0.0015" iyz="0.0" izz="0.0015"/>
-        </inertial>
-        <visual>
-            <origin xyz="0 0 0"
-                    rpy="0 0 0"/>
-            <geometry>
-                <mesh filename="package://niryo_robot_description/meshes/ned2/collada/shoulder_link.dae"/>
-            </geometry>
-        </visual>
-        <collision>
-            <origin xyz="0 0 0"
-                    rpy="0 0 0"/>
-            <geometry>
-                <mesh filename="package://niryo_robot_description/meshes/ned2/stl/shoulder_link.stl"/>
-            </geometry>
-        </collision>
-    </link>
-    <joint name="joint_2"
-           type="revolute">
-        <origin xyz="0 0 0.065"
-                rpy="${PI/2} ${-PI/2} 0"/>
+    <joint name="joint_2" type="revolute">
+        <origin xyz="0 0 0.065" rpy="${PI/2} ${-PI/2} 0"/>
         <parent link="shoulder_link"/>
         <child link="arm_link"/>
@@ -74,30 +209,6 @@
                upper="${(limit_up_arm_rotation - safety_pos_margin) * deg_to_rad}"/>
     </joint>
-    <link name="arm_link">
-        <inertial>
-            <origin xyz="0.116485160625991 -0.00141190194997476 -0.00338105503061108"
-                    rpy="0 0 0"/>
-            <mass value="0.513332159226246"/>
-            <inertia ixx="0.0015" ixy="0.0" ixz="0.0" iyy="0.0015" iyz="0.0" izz="0.0015"/>
-        </inertial>
-        <visual>
-            <origin xyz="0 0 0"
-                    rpy="0 0 0"/>
-            <geometry>
-                <mesh filename="package://niryo_robot_description/meshes/ned2/collada/arm_link.dae"/>
-            </geometry>
-        </visual>
-        <collision>
-            <origin xyz="0 0 0"
-                    rpy="0 0 0"/>
-            <geometry>
-                <mesh filename="package://niryo_robot_description/meshes/ned2/stl/arm_link.stl"/>
-            </geometry>
-        </collision>
-    </link>
-    <joint name="joint_3"
-           type="revolute">
-        <origin xyz="0.221 -0.012 0"
-                rpy="0 0 ${-PI/2}"/>
+    <joint name="joint_3" type="revolute">
+        <origin xyz="0.221 -0.012 0" rpy="0 0 ${-PI/2}"/>
         <parent link="arm_link"/>
         <child link="elbow_link"/>
@@ -106,30 +217,6 @@
                upper="${(limit_up_elbow_rotation - safety_pos_margin) * deg_to_rad}"/>
     </joint>
-    <link name="elbow_link">
-        <inertial>
-            <origin xyz="0.00840548736069937 0.0235132719991579 0.00139784606943909"
-                    rpy="0 0 0"/>
-            <mass value="0.201038841892435"/>
-            <inertia ixx="0.0015" ixy="0.0" ixz="0.0" iyy="0.0015" iyz="0.0" izz="0.0015"/>
-        </inertial>
-        <visual>
-            <origin xyz="0 0 0"
-                    rpy="0 0 0"/>
-            <geometry>
-                <mesh filename="package://niryo_robot_description/meshes/ned2/collada/elbow_link.dae"/>
-            </geometry>
-        </visual>
-        <collision>
-            <origin xyz="0 0 0"
-                    rpy="0 0 0"/>
-            <geometry>
-                <mesh filename="package://niryo_robot_description/meshes/ned2/stl/elbow_link.stl"/>
-            </geometry>
-        </collision>
-    </link>
-    <joint name="joint_4"
-           type="revolute">
-        <origin xyz="0.047 0.0325 0"
-                rpy="0 ${PI/2} 0"/>
+    <joint name="joint_4" type="revolute">
+        <origin xyz="0.065 0.0325 0" rpy="0 ${PI/2} 0"/>
         <parent link="elbow_link"/>
         <child link="forearm_link"/>
@@ -138,114 +225,25 @@
                upper="${(limit_up_forearm_rotation - safety_pos_margin) * deg_to_rad}"/>
     </joint>
-    <link name="forearm_link">
-        <inertial>
-            <origin xyz="-0.00811345462189901 -0.000135618649565461 0.107402242790047"
-                    rpy="0 0 0"/>
-            <mass value="0.203543862275952"/>
-            <inertia ixx="0.0015" ixy="0.0" ixz="0.0" iyy="0.0015" iyz="0.0" izz="0.0015"/>
-        </inertial>
-        <visual>
-            <origin xyz="0 0 0"
-                    rpy="0 0 0"/>
-            <geometry>
-                <mesh filename="package://niryo_robot_description/meshes/ned2/collada/forearm_link.dae"/>
-            </geometry>
-        </visual>
-        <collision>
-            <origin xyz="0 0 0"
-                    rpy="0 0 0"/>
-            <geometry>
-                <mesh filename="package://niryo_robot_description/meshes/ned2/stl/forearm_link.stl"/>
-            </geometry>
-        </collision>
-    </link>
-    <!-- add collision for the motor of joint 5 -->
-    <link name="joint5_motor">
-        <inertial>
-            <origin xyz="-0.00811345462189901 -0.000135618649565461 0.107402242790047"
-                    rpy="0 0 0"/>
-            <mass value="0.203543862275952"/>
-            <inertia ixx="0.0015" ixy="0.0" ixz="0.0" iyy="0.0015" iyz="0.0" izz="0.0015"/>
-        </inertial>
-        <collision>
-            <origin xyz="-0.045 0.0 0.1765"
-                    rpy="0 0 0"/>
-            <geometry>
-                <!-- <box size="0.03 0.03 0.046"/>  -->
-                <box size="0.0435 0.0285 0.0465"/>
-            </geometry>
-        </collision>
-    </link>
-    <joint name="joint_test"
-           type="fixed">
-        <origin xyz="0 0 0"
-                rpy="0 0 0"/>
+    <joint name="joint_5" type="revolute">
+        <origin xyz="0 0 0.17" rpy="${PI} ${-PI/2} ${PI}"/>
+        <parent link="forearm_link"/>
+        <child link="wrist_link"/>
+        <axis xyz="0 0 1"/>
+        <limit effort="6.0" velocity="2.0" lower="${(limit_low_wrist_rotation + safety_pos_margin) * deg_to_rad}"
+               upper="${(limit_up_wrist_rotation - safety_pos_margin) * deg_to_rad}"/>
+    </joint>
+    <joint name="joint_6" type="revolute">
+        <origin xyz="0.0197 0.00925 0" rpy="0 ${PI/2} 0"/>
+        <parent link="wrist_link"/>
+        <child link="hand_link"/>
+        <axis xyz="0 0 1"/>
+        <limit effort="5.0" velocity="2.0" lower="${(limit_low_hand_rotation + safety_pos_margin) * deg_to_rad}"
+               upper="${(limit_up_hand_rotation - safety_pos_margin) * deg_to_rad}"/>
+    </joint>
+    <joint name="joint_test" type="fixed">
+        <origin xyz="-0.03 0 0.158" rpy="0 -${PI/2} 0"/>
         <parent link="forearm_link"/>
         <child link="joint5_motor"/>
     </joint>
-    <joint name="joint_5"
-           type="revolute">
-        <origin xyz="0 0 0.188"
-                rpy="${PI} ${-PI/2} ${PI}"/>
-        <parent link="forearm_link"/>
-        <child link="wrist_link"/>
-        <axis xyz="0 0 1"/>
-        <limit effort="6.0" velocity="2.0" lower="${(limit_low_wrist_rotation + safety_pos_margin) * deg_to_rad}"
-               upper="${(limit_up_wrist_rotation - safety_pos_margin) * deg_to_rad}"/>
-    </joint>
-    <link name="wrist_link">
-        <inertial>
-            <origin xyz="-0.0193227036920796 -0.00157014407079775 0.000275751023741896"
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
File: niryo_robot_description/urdf/ned2/niryo_ned2_camera.urdf.xacro (robot description, xacro)
@@ -10,5 +10,5 @@
     <joint name="camera_joint" type="fixed">
         <axis xyz="0 0 1"/>
-        <origin xyz="0 ${cameraHeight/2 + 0.02} 0" rpy="${PI/2} 0 0"/>
+        <origin xyz="0 ${cameraHeight/2 + 0.02} 0" rpy="${PI/2} 0 ${deg_to_rad*10}"/>
         <parent link="wrist_link"/>
         <child link="camera_link"/>

File: niryo_robot_description/urdf/ned2/niryo_ned2_gripper1_n_camera.urdf.xacro (robot description, xacro)
@@ -17,5 +17,5 @@
         <child link="base_gripper_1"/>
         <origin
-                xyz="0 0 0.005"
+                xyz="0.005 0 0.005"
                 rpy="0 ${PI/2} ${PI/2}"/>
     </joint>

Commit message: fix link collisions + roslaunch

File: niryo_robot_description/urdf/ned2/niryo_ned2.urdf.xacro (robot description, xacro)
@@ -246,4 +246,70 @@
         <child link="joint5_motor"/>
     </joint>
+    <link name="tool_link">
+    </link>
+    <!-- Joints -->
+    <joint name="joint_world" type="fixed">
+        <parent link="world"/>
+        <child link="base_link"/>
+        <origin xyz="0 0 0" rpy="0 0 0"/>
+    </joint>
+    <joint name="joint_led_ring" type="fixed">
+        <parent link="world"/>
+        <child link="led_ring_link"/>
+        <origin xyz="0 0 0.0923" rpy="0 0 ${PI/2}"/>
+    </joint>
+    <joint name="joint_1" type="revolute">
+        <origin xyz="0 3.7961E-05 0.1013" rpy="0 0 0"/>
+        <parent link="base_link"/>
+        <child link="shoulder_link"/>
+        <axis xyz="0 0 1"/>
+        <limit effort="10.0" velocity="10.0" lower="${(limit_low_shoulder_rotation + safety_pos_margin) * deg_to_rad}"
+               upper="${(limit_up_shoulder_rotation - safety_pos_margin) * deg_to_rad}"/>
+    </joint>
+    <joint name="joint_2" type="revolute">
+        <origin xyz="0 0 0.065" rpy="${PI/2} ${-PI/2} 0"/>
+        <parent link="shoulder_link"/>
+        <child link="arm_link"/>
+        <axis xyz="0 0 1"/>
+        <limit effort="10.0" velocity="8.0" lower="${(limit_low_arm_rotation + safety_pos_margin) * deg_to_rad}"
+               upper="${(limit_up_arm_rotation - safety_pos_margin) * deg_to_rad}"/>
+    </joint>
+    <joint name="joint_3" type="revolute">
+        <origin xyz="0.221 -0.012 0" rpy="0 0 ${-PI/2}"/>
+        <parent link="arm_link"/>
+        <child link="elbow_link"/>
+        <axis xyz="0 0 1"/>
+        <limit effort="7.0" velocity="8.0" lower="${(limit_low_elbow_rotation + safety_pos_margin) * deg_to_rad}"
+               upper="${(limit_up_elbow_rotation - safety_pos_margin) * deg_to_rad}"/>
+    </joint>
+    <joint name="joint_4" type="revolute">
+        <origin xyz="0.065 0.0325 0" rpy="0 ${PI/2} 0"/>
+        <parent link="elbow_link"/>
+        <child link="forearm_link"/>
+        <axis xyz="0 0 1"/>
+        <limit effort="7.0" velocity="2.0" lower="${(limit_low_forearm_rotation + safety_pos_margin) * deg_to_rad}"
+               upper="${(limit_up_forearm_rotation - safety_pos_margin) * deg_to_rad}"/>
+    </joint>
+    <joint name="joint_5" type="revolute">
+        <origin xyz="0 0 0.17" rpy="${PI} ${-PI/2} ${PI}"/>
+        <parent link="forearm_link"/>
+        <child link="wrist_link"/>
+        <axis xyz="0 0 1"/>
+        <limit effort="6.0" velocity="2.0" lower="${(limit_low_wrist_rotation + safety_pos_margin) * deg_to_rad}"
+               upper="${(limit_up_wrist_rotation - safety_pos_margin) * deg_to_rad}"/>
+    </joint>
+    <joint name="joint_6" type="revolute">
+        <origin xyz="0.0197 0.00925 0" rpy="0 ${PI/2} 0"/>
+        <parent link="wrist_link"/>
+        <child link="hand_link"/>
+        <axis xyz="0 0 1"/>
+        <limit effort="5.0" velocity="2.0" lower="${(limit_low_hand_rotation + safety_pos_margin) * deg_to_rad}"
+               upper="${(limit_up_hand_rotation - safety_pos_margin) * deg_to_rad}"/>
+    </joint>
+    <joint name="joint_test" type="fixed">
+        <origin xyz="-0.03 0 0.158" rpy="0 -${PI/2} 0"/>
+        <parent link="forearm_link"/>
+        <child link="joint5_motor"/>
+    </joint>
     <joint name="hand_tool_joint" type="fixed">
         <parent link="hand_link"/>
