Commit message: Fix urdf + end effector panel python

File: niryo_robot_description/urdf/ned2/niryo_ned2.urdf.xacro (robot description, xacro)
@@ -246,70 +246,4 @@
         <child link="joint5_motor"/>
     </joint>
-    <link name="tool_link">
-    </link>
-    <!-- Joints -->
-    <joint name="joint_world" type="fixed">
-        <parent link="world"/>
-        <child link="base_link"/>
-        <origin xyz="0 0 0" rpy="0 0 0"/>
-    </joint>
-    <joint name="joint_led_ring" type="fixed">
-        <parent link="world"/>
-        <child link="led_ring_link"/>
-        <origin xyz="0 0 0.0923" rpy="0 0 ${PI/2}"/>
-    </joint>
-    <joint name="joint_1" type="revolute">
-        <origin xyz="0 3.7961E-05 0.1013" rpy="0 0 0"/>
-        <parent link="base_link"/>
-        <child link="shoulder_link"/>
-        <axis xyz="0 0 1"/>
-        <limit effort="10.0" velocity="10.0" lower="${(limit_low_shoulder_rotation + safety_pos_margin) * deg_to_rad}"
-               upper="${(limit_up_shoulder_rotation - safety_pos_margin) * deg_to_rad}"/>
-    </joint>
-    <joint name="joint_2" type="revolute">
-        <origin xyz="0 0 0.065" rpy="${PI/2} ${-PI/2} 0"/>
-        <parent link="shoulder_link"/>
-        <child link="arm_link"/>
-        <axis xyz="0 0 1"/>
-        <limit effort="10.0" velocity="8.0" lower="${(limit_low_arm_rotation + safety_pos_margin) * deg_to_rad}"
-               upper="${(limit_up_arm_rotation - safety_pos_margin) * deg_to_rad}"/>
-    </joint>
-    <joint name="joint_3" type="revolute">
-        <origin xyz="0.221 -0.012 0" rpy="0 0 ${-PI/2}"/>
-        <parent link="arm_link"/>
-        <child link="elbow_link"/>
-        <axis xyz="0 0 1"/>
-        <limit effort="7.0" velocity="8.0" lower="${(limit_low_elbow_rotation + safety_pos_margin) * deg_to_rad}"
-               upper="${(limit_up_elbow_rotation - safety_pos_margin) * deg_to_rad}"/>
-    </joint>
-    <joint name="joint_4" type="revolute">
-        <origin xyz="0.065 0.0325 0" rpy="0 ${PI/2} 0"/>
-        <parent link="elbow_link"/>
-        <child link="forearm_link"/>
-        <axis xyz="0 0 1"/>
-        <limit effort="7.0" velocity="2.0" lower="${(limit_low_forearm_rotation + safety_pos_margin) * deg_to_rad}"
-               upper="${(limit_up_forearm_rotation - safety_pos_margin) * deg_to_rad}"/>
-    </joint>
-    <joint name="joint_5" type="revolute">
-        <origin xyz="0 0 0.17" rpy="${PI} ${-PI/2} ${PI}"/>
-        <parent link="forearm_link"/>
-        <child link="wrist_link"/>
-        <axis xyz="0 0 1"/>
-        <limit effort="6.0" velocity="2.0" lower="${(limit_low_wrist_rotation + safety_pos_margin) * deg_to_rad}"
-               upper="${(limit_up_wrist_rotation - safety_pos_margin) * deg_to_rad}"/>
-    </joint>
-    <joint name="joint_6" type="revolute">
-        <origin xyz="0.0197 0.00925 0" rpy="0 ${PI/2} 0"/>
-        <parent link="wrist_link"/>
-        <child link="hand_link"/>
-        <axis xyz="0 0 1"/>
-        <limit effort="5.0" velocity="2.0" lower="${(limit_low_hand_rotation + safety_pos_margin) * deg_to_rad}"
-               upper="${(limit_up_hand_rotation - safety_pos_margin) * deg_to_rad}"/>
-    </joint>
-    <joint name="joint_test" type="fixed">
-        <origin xyz="-0.03 0 0.158" rpy="0 -${PI/2} 0"/>
-        <parent link="forearm_link"/>
-        <child link="joint5_motor"/>
-    </joint>
     <joint name="hand_tool_joint" type="fixed">
         <parent link="hand_link"/>

Commit message: Fix ned2 urdf

File: niryo_robot_description/urdf/ned2/niryo_ned2.urdf.xacro (robot description, xacro)
@@ -127,8 +127,7 @@
     <link name="joint5_motor">
         <inertial>
-            <origin xyz="-0.00811345462189901 -0.000135618649565461 0.107402242790047"
-                    rpy="0 0 0"/>
+            <origin xyz="0 0 0.015" rpy="0 0 0"/>
             <mass value="0.203543862275952"/>
-            <inertia ixx="0.0015" ixy="0.0" ixz="0.0" iyy="0.0015" iyz="0.0" izz="0.0015"/>
+            <inertia ixx="0.000" ixy="0.0" ixz="0.0" iyy="0.000" iyz="0.0" izz="0.0015"/>
         </inertial>
         <collision>
@@ -188,9 +187,4 @@
         <origin xyz="0 0 0" rpy="0 0 0"/>
     </joint>
-    <joint name="joit_led_ring" type="fixed">
-        <parent link="world"/>
-        <child link="led_ring_link"/>
-        <origin xyz="0 0 0.0923" rpy="0 0 0"/>
-    </joint>
     <joint name="joint_1" type="revolute">
         <origin xyz="0 3.7961E-05 0.1013" rpy="0 0 0"/>
@@ -218,5 +212,5 @@
     </joint>
     <joint name="joint_4" type="revolute">
-        <origin xyz="0.065 0.0325 0" rpy="0 ${PI/2} 0"/>
+        <origin xyz="0. 0.0325 0" rpy="0 ${PI/2} 0"/>
         <parent link="elbow_link"/>
         <child link="forearm_link"/>
@@ -241,4 +235,9 @@
                upper="${(limit_up_hand_rotation - safety_pos_margin) * deg_to_rad}"/>
     </joint>
+    <joint name="hand_tool_joint" type="fixed">
+        <parent link="hand_link"/>
+        <child link="tool_link"/>
+        <origin xyz="0 0 ${distance_hand_tool}" rpy="${-PI/2} ${-PI/2} 0"/>
+    </joint>
     <joint name="joint_test" type="fixed">
         <origin xyz="-0.03 0 0.158" rpy="0 -${PI/2} 0"/>
@@ -246,8 +245,8 @@
         <child link="joint5_motor"/>
     </joint>
-    <joint name="hand_tool_joint" type="fixed">
-        <parent link="hand_link"/>
-        <child link="tool_link"/>
-        <origin xyz="0 0 ${distance_hand_tool}" rpy="${-PI/2} ${-PI/2} 0"/>
+    <joint name="joint_led_ring" type="fixed">
+        <parent link="world"/>
+        <child link="led_ring_link"/>
+        <origin xyz="0 0 0.0923" rpy="0 0 0"/>
     </joint>
 </robot>

File: niryo_robot_description/urdf/ned2/without_mesh_niryo_ned2.urdf.xacro (robot description, xacro)
@@ -5,13 +5,7 @@
     <!-- Links -->
     <link name="world"/>
-    <joint name="joint_world" type="fixed">
-        <parent link="world"/>
-        <child link="base_link"/>
-        <origin xyz="0 0 0" rpy="0 0 0"/>
-    </joint>
     <link name="base_link">
         <collision>
-            <origin xyz="0 0 0"
-                    rpy="0 0 0"/>
+            <origin xyz="0 0 0" rpy="0 0 0"/>
             <geometry>
                 <mesh filename="package://niryo_robot_description/meshes/ned2/stl/base_link.stl"/>
@@ -19,18 +13,7 @@
         </collision>
     </link>
-    <joint name="joint_1"
-           type="revolute">
-        <origin xyz="0 0 0.1065"
-                rpy="0 0 0"/>
-        <parent link="base_link"/>
-        <child link="shoulder_link"/>
-        <axis xyz="0 0 1"/>
-        <limit effort="10.0" velocity="2.2" lower="${(limit_low_shoulder_rotation + safety_pos_margin) * deg_to_rad}"
-               upper="${(limit_up_shoulder_rotation - safety_pos_margin) * deg_to_rad}"/>
-    </joint>
     <link name="shoulder_link">
         <collision>
-            <origin xyz="0 0 0"
-                    rpy="0 0 0"/>
+            <origin xyz="0 0 0" rpy="0 0 0"/>
             <geometry>
                 <mesh filename="package://niryo_robot_description/meshes/ned2/stl/shoulder_link.stl"/>
@@ -38,18 +21,7 @@
         </collision>
     </link>
-    <joint name="joint_2"
-           type="revolute">
-        <origin xyz="0 0 0.065"
-                rpy="${PI/2} ${-PI/2} 0"/>
-        <parent link="shoulder_link"/>
-        <child link="arm_link"/>
-        <axis xyz="0 0 1"/>
-        <limit effort="10.0" velocity="2.2" lower="${(limit_low_arm_rotation + safety_pos_margin) * deg_to_rad}"
-               upper="${(limit_up_arm_rotation - safety_pos_margin) * deg_to_rad}"/>
-    </joint>
     <link name="arm_link">
         <collision>
-            <origin xyz="0 0 0"
-                    rpy="0 0 0"/>
+            <origin xyz="0 0 0" rpy="0 0 0"/>
             <geometry>
                 <mesh filename="package://niryo_robot_description/meshes/ned2/stl/arm_link.stl"/>
@@ -57,18 +29,7 @@
         </collision>
     </link>
-    <joint name="joint_3"
-           type="revolute">
-        <origin xyz="0.221 -0.012 0"
-                rpy="0 0 ${-PI/2}"/>
-        <parent link="arm_link"/>
-        <child link="elbow_link"/>
-        <axis xyz="0 0 1"/>
-        <limit effort="7.0" velocity="2.0" lower="${(limit_low_elbow_rotation + safety_pos_margin) * deg_to_rad}"
-               upper="${(limit_up_elbow_rotation - safety_pos_margin) * deg_to_rad}"/>
-    </joint>
     <link name="elbow_link">
         <collision>
-            <origin xyz="0 0 0"
-                    rpy="0 0 0"/>
+            <origin xyz="0 0 0" rpy="0 0 0"/>
             <geometry>
                 <mesh filename="package://niryo_robot_description/meshes/ned2/stl/elbow_link.stl"/>
@@ -76,18 +37,7 @@
         </collision>
     </link>
-    <joint name="joint_4"
-           type="revolute">
-        <origin xyz="0.047 0.0325 0"
-                rpy="0 ${PI/2} 0"/>
-        <parent link="elbow_link"/>
-        <child link="forearm_link"/>
-        <axis xyz="0 0 1"/>
-        <limit effort="7.0" velocity="2.0" lower="${(limit_low_forearm_rotation + safety_pos_margin) * deg_to_rad}"
-               upper="${(limit_up_forearm_rotation - safety_pos_margin) * deg_to_rad}"/>
-    </joint>
     <link name="forearm_link">
         <collision>
-            <origin xyz="0 0 0"
-                    rpy="0 0 0"/>
+            <origin xyz="0 0 0" rpy="0 0 0"/>
             <geometry>
                 <mesh filename="package://niryo_robot_description/meshes/ned2/stl/forearm_link.stl"/>
@@ -98,22 +48,70 @@
     <link name="joint5_motor">
         <collision>
-            <origin xyz="-0.045 0.0 0.1765"
-                    rpy="0 0 0"/>
+            <origin xyz="0 0 0.015" rpy="0 0 0"/>
             <geometry>
-                <box size="0.0435 0.0285 0.0465"/>
+                <box size="0.047 0.0285 0.03"/>
             </geometry>
         </collision>
     </link>
-    <joint name="joint_test"
-           type="fixed">
-        <origin xyz="0 0 0"
-                rpy="0 0 0"/>
-        <parent link="forearm_link"/>
-        <child link="joint5_motor"/>
+    <link name="wrist_link">
+        <collision>
+            <origin xyz="0 0 0" rpy="0 0 0"/>
+            <geometry>
+                <mesh filename="package://niryo_robot_description/meshes/ned2/stl/wrist_link.stl"/>
+            </geometry>
+        </collision>
+    </link>
+    <link name="hand_link">
+        <collision>
+            <origin xyz="0 0 0"  rpy="0 0 0"/>
+            <geometry>
+                <mesh filename="package://niryo_robot_description/meshes/ned2/stl/hand_link.stl"/>
+            </geometry>
+        </collision>
+    </link>
+    <link name="tool_link">
+    </link>
+    <link name="led_ring_link">
+    </link>
+    <!-- Joints -->
+    <joint name="joint_world" type="fixed">
+        <parent link="world"/>
+        <child link="base_link"/>
+        <origin xyz="0 0 0" rpy="0 0 0"/>
     </joint>
-    <joint name="joint_5"
-           type="revolute">
-        <origin xyz="0 0 0.188"
-                rpy="${PI} ${-PI/2} ${PI}"/>
+    <joint name="joint_1" type="revolute">
+        <origin xyz="0 3.7961E-05 0.1013" rpy="0 0 0"/>
+        <parent link="base_link"/>
+        <child link="shoulder_link"/>
+        <axis xyz="0 0 1"/>
+        <limit effort="10.0" velocity="2.2" lower="${(limit_low_shoulder_rotation + safety_pos_margin) * deg_to_rad}"
+               upper="${(limit_up_shoulder_rotation - safety_pos_margin) * deg_to_rad}"/>
+    </joint>
+    <joint name="joint_2" type="revolute">
+        <origin xyz="0 0 0.065" rpy="${PI/2} ${-PI/2} 0"/>
+        <parent link="shoulder_link"/>
+        <child link="arm_link"/>
+        <axis xyz="0 0 1"/>
+        <limit effort="10.0" velocity="2.2" lower="${(limit_low_arm_rotation + safety_pos_margin) * deg_to_rad}"
+               upper="${(limit_up_arm_rotation - safety_pos_margin) * deg_to_rad}"/>
+    </joint>
+    <joint name="joint_3" type="revolute">
+        <origin xyz="0.221 -0.012 0" rpy="0 0 ${-PI/2}"/>
+        <parent link="arm_link"/>
+        <child link="elbow_link"/>
+        <axis xyz="0 0 1"/>
+        <limit effort="7.0" velocity="2.0" lower="${(limit_low_elbow_rotation + safety_pos_margin) * deg_to_rad}"
+               upper="${(limit_up_elbow_rotation - safety_pos_margin) * deg_to_rad}"/>
+    </joint>
+    <joint name="joint_4" type="revolute">
+        <origin xyz="0.065 0.0325 0" rpy="0 ${PI/2} 0"/>
+        <parent link="elbow_link"/>
+        <child link="forearm_link"/>
+        <axis xyz="0 0 1"/>
+        <limit effort="7.0" velocity="2.0" lower="${(limit_low_forearm_rotation + safety_pos_margin) * deg_to_rad}"
+               upper="${(limit_up_forearm_rotation - safety_pos_margin) * deg_to_rad}"/>
+    </joint>
+    <joint name="joint_5" type="revolute">
+        <origin xyz="0 0 0.17" rpy="${PI} ${-PI/2} ${PI}"/>
         <parent link="forearm_link"/>
         <child link="wrist_link"/>
@@ -122,17 +120,6 @@
                upper="${(limit_up_wrist_rotation - safety_pos_margin) * deg_to_rad}"/>
     </joint>
-    <link name="wrist_link">
-        <collision>
-            <origin xyz="0 0 0"
-                    rpy="0 0 0"/>
-            <geometry>
-                <mesh filename="package://niryo_robot_description/meshes/ned2/stl/wrist_link.stl"/>
-            </geometry>
-        </collision>
-    </link>
-    <joint name="joint_6"
-           type="revolute">
-        <origin xyz="0.0197 0.00925 0"
-                rpy="0 ${PI/2} 0"/>
+    <joint name="joint_6" type="revolute">
+        <origin xyz="0.0197 0.00925 0" rpy="0 ${PI/2} 0"/>
         <parent link="wrist_link"/>
         <child link="hand_link"/>
@@ -141,13 +128,4 @@
                upper="${(limit_up_hand_rotation - safety_pos_margin) * deg_to_rad}"/>
     </joint>
-    <link name="hand_link">
-        <collision>
-            <origin xyz="0 0 0"
-                    rpy="0 0 0"/>
-            <geometry>
-                <mesh filename="package://niryo_robot_description/meshes/ned2/stl/hand_link.stl"/>
-            </geometry>
-        </collision>
-    </link>
     <joint name="hand_tool_joint" type="fixed">
         <parent link="hand_link"/>
@@ -155,8 +133,9 @@
         <origin xyz="0 0 ${distance_hand_tool}" rpy="${-PI/2} ${-PI/2} 0"/>
     </joint>
-    <link name="tool_link">
-    </link>
-    <link name="led_ring_link">
-    </link>
+    <joint name="joint_test" type="fixed">
+        <origin xyz="-0.03 0 0.158" rpy="0 -${PI/2} 0"/>
+        <parent link="forearm_link"/>
+        <child link="joint5_motor"/>
+    </joint>
     <joint name="joint_led_ring" type="fixed">
         <parent link="world"/>

Commit message: fix urdf ned2

File: niryo_robot_description/urdf/ned2/niryo_ned2.urdf.xacro (robot description, xacro)
@@ -212,5 +212,5 @@
     </joint>
     <joint name="joint_4" type="revolute">
-        <origin xyz="0. 0.0325 0" rpy="0 ${PI/2} 0"/>
+        <origin xyz="0.065 0.0325 0" rpy="0 ${PI/2} 0"/>
         <parent link="elbow_link"/>
         <child link="forearm_link"/>

Commit message: Tickets val

File: niryo_robot_description/urdf/ned2/niryo_ned2.urdf.xacro (robot description, xacro)
@@ -127,8 +127,7 @@
     <link name="joint5_motor">
         <inertial>
-            <origin xyz="-0.00811345462189901 -0.000135618649565461 0.107402242790047"
-                    rpy="0 0 0"/>
+            <origin xyz="0 0 0.015" rpy="0 0 0"/>
             <mass value="0.203543862275952"/>
-            <inertia ixx="0.0015" ixy="0.0" ixz="0.0" iyy="0.0015" iyz="0.0" izz="0.0015"/>
+            <inertia ixx="0.000" ixy="0.0" ixz="0.0" iyy="0.000" iyz="0.0" izz="0.0015"/>
         </inertial>
         <collision>
@@ -188,9 +187,4 @@
         <origin xyz="0 0 0" rpy="0 0 0"/>
     </joint>
-    <joint name="joit_led_ring" type="fixed">
-        <parent link="world"/>
-        <child link="led_ring_link"/>
-        <origin xyz="0 0 0.0923" rpy="0 0 0"/>
-    </joint>
     <joint name="joint_1" type="revolute">
         <origin xyz="0 3.7961E-05 0.1013" rpy="0 0 0"/>
@@ -241,4 +235,9 @@
                upper="${(limit_up_hand_rotation - safety_pos_margin) * deg_to_rad}"/>
     </joint>
+    <joint name="hand_tool_joint" type="fixed">
+        <parent link="hand_link"/>
+        <child link="tool_link"/>
+        <origin xyz="0 0 ${distance_hand_tool}" rpy="${-PI/2} ${-PI/2} 0"/>
+    </joint>
     <joint name="joint_test" type="fixed">
         <origin xyz="-0.03 0 0.158" rpy="0 -${PI/2} 0"/>
@@ -246,8 +245,8 @@
         <child link="joint5_motor"/>
     </joint>
-    <joint name="hand_tool_joint" type="fixed">
-        <parent link="hand_link"/>
-        <child link="tool_link"/>
-        <origin xyz="0 0 ${distance_hand_tool}" rpy="${-PI/2} ${-PI/2} 0"/>
+    <joint name="joint_led_ring" type="fixed">
+        <parent link="world"/>
+        <child link="led_ring_link"/>
+        <origin xyz="0 0 0.0923" rpy="0 0 0"/>
     </joint>
 </robot>

Commit message: Fix ned2 urdf inertia for gazebo simulation

File: niryo_robot_description/urdf/ned2/niryo_ned2.urdf.xacro (robot description, xacro)
@@ -129,5 +129,5 @@
             <origin xyz="0 0 0.015" rpy="0 0 0"/>
             <mass value="0.203543862275952"/>
-            <inertia ixx="0.000" ixy="0.0" ixz="0.0" iyy="0.000" iyz="0.0" izz="0.0015"/>
+            <inertia ixx="0.0015" ixy="0.0" ixz="0.0" iyy="0.0015" iyz="0.0" izz="0.0015"/>
         </inertial>
         <collision>

Commit message: Ned2 beta

File: niryo_robot_description/urdf/ned2/niryo_ned2.urdf.xacro (robot description, xacro)
@@ -127,6 +127,5 @@
     <link name="joint5_motor">
         <inertial>
-            <origin xyz="-0.00811345462189901 -0.000135618649565461 0.107402242790047"
-                    rpy="0 0 0"/>
+            <origin xyz="0 0 0.015" rpy="0 0 0"/>
             <mass value="0.203543862275952"/>
             <inertia ixx="0.0015" ixy="0.0" ixz="0.0" iyy="0.0015" iyz="0.0" izz="0.0015"/>
@@ -188,9 +187,4 @@
         <origin xyz="0 0 0" rpy="0 0 0"/>
     </joint>
-    <joint name="joit_led_ring" type="fixed">
-        <parent link="world"/>
-        <child link="led_ring_link"/>
-        <origin xyz="0 0 0.0923" rpy="0 0 0"/>
-    </joint>
     <joint name="joint_1" type="revolute">
         <origin xyz="0 3.7961E-05 0.1013" rpy="0 0 0"/>
@@ -241,4 +235,9 @@
                upper="${(limit_up_hand_rotation - safety_pos_margin) * deg_to_rad}"/>
     </joint>
+    <joint name="hand_tool_joint" type="fixed">
+        <parent link="hand_link"/>
+        <child link="tool_link"/>
+        <origin xyz="0 0 ${distance_hand_tool}" rpy="${-PI/2} ${-PI/2} 0"/>
+    </joint>
     <joint name="joint_test" type="fixed">
         <origin xyz="-0.03 0 0.158" rpy="0 -${PI/2} 0"/>
@@ -246,8 +245,8 @@
         <child link="joint5_motor"/>
     </joint>
-    <joint name="hand_tool_joint" type="fixed">
-        <parent link="hand_link"/>
-        <child link="tool_link"/>
-        <origin xyz="0 0 ${distance_hand_tool}" rpy="${-PI/2} ${-PI/2} 0"/>
+    <joint name="joint_led_ring" type="fixed">
+        <parent link="world"/>
+        <child link="led_ring_link"/>
+        <origin xyz="0 0 0.0923" rpy="0 0 0"/>
     </joint>
 </robot>
