Commit message: SN-278: Add ned3 drivers, registers & config files

File: niryo_robot_description/urdf/ned2/niryo_ned2.urdf.xacro (robot description, xacro)
@@ -47,5 +47,5 @@
         </inertial>
         <visual>
-            <origin xyz="0 0 0" rpy="0 0 0"/>
+            <origin xyz="0 0 0" rpy="0 0 ${-PI/2}"/>
             <geometry>
                 <mesh filename="package://niryo_robot_description/meshes/ned2/collada/shoulder_link.dae"/>
@@ -53,5 +53,5 @@
         </visual>
         <collision>
-            <origin xyz="0 0 0" rpy="0 0 0"/>
+            <origin xyz="0 0 0" rpy="0 0 ${-PI/2}"/>
             <geometry>
                 <mesh filename="package://niryo_robot_description/meshes/ned2/stl/shoulder_link.stl"/>
@@ -86,5 +86,5 @@
         </inertial>
         <visual>
-            <origin xyz="0 0 0" rpy="0 ${PI} 0"/>
+            <origin xyz="0 0 0" rpy="0 ${PI} ${-PI/2}"/>
             <geometry>
                 <mesh filename="package://niryo_robot_description/meshes/ned2/collada/elbow_link.dae"/>
@@ -92,5 +92,5 @@
         </visual>
         <collision>
-            <origin xyz="0 0 0" rpy="0 ${PI} 0"/>
+            <origin xyz="0 0 0" rpy="0 ${PI} ${-PI/2}"/>
             <geometry>
                 <mesh filename="package://niryo_robot_description/meshes/ned2/stl/elbow_link.stl"/>
@@ -106,5 +106,5 @@
         </inertial>
         <visual>
-            <origin xyz="0 0 0" rpy="0 0 0"/>
+            <origin xyz="0 0 0" rpy="0 0 ${-PI/2}"/>
             <geometry>
                 <mesh filename="package://niryo_robot_description/meshes/ned2/collada/forearm_link.dae"/>
@@ -112,5 +112,5 @@
         </visual>
         <collision>
-            <origin xyz="0 0 0" rpy="0 0 0"/>
+            <origin xyz="0 0 0" rpy="0 0 ${-PI/2}"/>
             <geometry>
                 <mesh filename="package://niryo_robot_description/meshes/ned2/stl/forearm_link.stl"/>
@@ -140,5 +140,5 @@
         <visual>
             <origin xyz="0 0 0"
-                    rpy="0 0 0"/>
+                    rpy="0 0 ${-PI/2}"/>
             <geometry>
                 <mesh filename="package://niryo_robot_description/meshes/ned2/collada/wrist_link.dae"/>
@@ -147,5 +147,5 @@
         <collision>
             <origin xyz="0 0 0"
-                    rpy="0 0 0"/>
+                    rpy="0 0 ${-PI/2}"/>
             <geometry>
                 <mesh filename="package://niryo_robot_description/meshes/ned2/stl/wrist_link.stl"/>
@@ -160,5 +160,5 @@
         </inertial>
         <visual>
-            <origin xyz="0 0 0" rpy="0 0 0"/>
+            <origin xyz="0 0 0" rpy="0 0 ${-PI/2}"/>
             <geometry>
                 <mesh filename="package://niryo_robot_description/meshes/ned2/collada/hand_link.dae"/>
@@ -166,5 +166,5 @@
         </visual>
         <collision>
-            <origin xyz="0 0 0" rpy="0 0 0"/>
+            <origin xyz="0 0 0" rpy="0 0 ${-PI/2}"/>
             <geometry>
                 <mesh filename="package://niryo_robot_description/meshes/ned2/stl/hand_link.stl"/>
@@ -181,5 +181,5 @@
     </joint>
     <joint name="joint_1" type="revolute">
-        <origin xyz="0 0 0.1013" rpy="0 0 ${-PI/2}"/>
+        <origin xyz="0 0 0.1013" rpy="0 0 0"/>
         <parent link="base_link"/>
         <child link="shoulder_link"/>
@@ -189,5 +189,5 @@
     </joint>
     <joint name="joint_2" type="revolute">
-        <origin xyz="0 0 0.065" rpy="${PI/2} 0 ${PI/2}"/>
+        <origin xyz="0 0 0.065" rpy="${PI/2} 0 0"/>
         <parent link="shoulder_link"/>
         <child link="arm_link"/>
@@ -197,5 +197,5 @@
     </joint>
     <joint name="joint_3" type="revolute">
-        <origin xyz="0.012 0.221 0" rpy="0 0 0"/>
+        <origin xyz="0.012 0.221 0" rpy="0 0 ${PI/2}"/>
         <parent link="arm_link"/>
         <child link="elbow_link"/>
@@ -205,5 +205,5 @@
     </joint>
     <joint name="joint_4" type="revolute">
-        <origin xyz="0.065 0.0325 0" rpy="0 ${PI/2} 0"/>
+        <origin xyz="0.0325 -0.065 0" rpy="${PI/2} 0 0"/>
         <parent link="elbow_link"/>
         <child link="forearm_link"/>
@@ -213,5 +213,5 @@
     </joint>
     <joint name="joint_5" type="revolute">
-        <origin xyz="0 0 0.17" rpy="${PI} ${-PI/2} ${PI}"/>
+        <origin xyz="0 0 0.17" rpy="${-PI/2} 0 0"/>
         <parent link="forearm_link"/>
         <child link="wrist_link"/>
@@ -221,5 +221,5 @@
     </joint>
     <joint name="joint_6" type="revolute">
-        <origin xyz="0.0197 0.00925 0" rpy="0 ${PI/2} 0"/>
+        <origin xyz="0.00925 -0.0197 0" rpy="${PI/2} 0 0"/>
         <parent link="wrist_link"/>
         <child link="hand_link"/>
@@ -231,5 +231,5 @@
         <parent link="hand_link"/>
         <child link="tool_link"/>
-        <origin xyz="0 0 ${distance_hand_tool}" rpy="${-PI/2} ${-PI/2} 0"/>
+        <origin xyz="0 0 ${distance_hand_tool}" rpy="0 0 0"/>
     </joint>
     <!--

File: niryo_robot_description/urdf/ned2/without_mesh_niryo_ned2.urdf.xacro (robot description, xacro)
@@ -41,5 +41,5 @@
         </inertial>
         <collision>
-            <origin xyz="0 0 0" rpy="0 0 0"/>
+            <origin xyz="0 0 0" rpy="0 0 ${-PI/2}"/>
             <geometry>
                 <mesh filename="package://niryo_robot_description/meshes/ned2/stl/shoulder_link.stl"/>
@@ -68,5 +68,5 @@
         </inertial>
         <collision>
-            <origin xyz="0 0 0" rpy="0 ${PI} 0"/>
+            <origin xyz="0 0 0" rpy="0 ${PI} ${-PI/2}"/>
             <geometry>
                 <mesh filename="package://niryo_robot_description/meshes/ned2/stl/elbow_link.stl"/>
@@ -82,5 +82,5 @@
         </inertial>
         <collision>
-            <origin xyz="0 0 0" rpy="0 0 0"/>
+            <origin xyz="0 0 0" rpy="0 0 ${-PI/2}"/>
             <geometry>
                 <mesh filename="package://niryo_robot_description/meshes/ned2/stl/forearm_link.stl"/>
@@ -110,5 +110,5 @@
         <collision>
             <origin xyz="0 0 0"
-                    rpy="0 0 0"/>
+                    rpy="0 0 ${-PI/2}"/>
             <geometry>
                 <mesh filename="package://niryo_robot_description/meshes/ned2/stl/wrist_link.stl"/>
@@ -123,5 +123,5 @@
         </inertial>
         <collision>
-            <origin xyz="0 0 0" rpy="0 0 0"/>
+            <origin xyz="0 0 0" rpy="0 0 ${-PI/2}"/>
             <geometry>
                 <mesh filename="package://niryo_robot_description/meshes/ned2/stl/hand_link.stl"/>
@@ -138,5 +138,5 @@
     </joint>
     <joint name="joint_1" type="revolute">
-        <origin xyz="0 0 0.1013" rpy="0 0 ${-PI/2}"/>
+        <origin xyz="0 0 0.1013" rpy="0 0 0"/>
         <parent link="base_link"/>
         <child link="shoulder_link"/>
@@ -146,5 +146,5 @@
     </joint>
     <joint name="joint_2" type="revolute">
-        <origin xyz="0 0 0.065" rpy="${PI/2} 0 ${PI/2}"/>
+        <origin xyz="0 0 0.065" rpy="${PI/2} 0 0"/>
         <parent link="shoulder_link"/>
         <child link="arm_link"/>
@@ -154,5 +154,5 @@
     </joint>
     <joint name="joint_3" type="revolute">
-        <origin xyz="0.012 0.221 0" rpy="0 0 0"/>
+        <origin xyz="0.012 0.221 0" rpy="0 0 ${PI/2}"/>
         <parent link="arm_link"/>
         <child link="elbow_link"/>
@@ -162,5 +162,5 @@
     </joint>
     <joint name="joint_4" type="revolute">
-        <origin xyz="0.065 0.0325 0" rpy="0 ${PI/2} 0"/>
+        <origin xyz="0.0325 -0.065 0" rpy="${PI/2} 0 0"/>
         <parent link="elbow_link"/>
         <child link="forearm_link"/>
@@ -170,5 +170,5 @@
     </joint>
     <joint name="joint_5" type="revolute">
-        <origin xyz="0 0 0.17" rpy="${PI} ${-PI/2} ${PI}"/>
+        <origin xyz="0 0 0.17" rpy="${-PI/2} 0 0"/>
         <parent link="forearm_link"/>
         <child link="wrist_link"/>
@@ -178,5 +178,5 @@
     </joint>
     <joint name="joint_6" type="revolute">
-        <origin xyz="0.0197 0.00925 0" rpy="0 ${PI/2} 0"/>
+        <origin xyz="0.00925 -0.0197 0" rpy="${PI/2} 0 0"/>
         <parent link="wrist_link"/>
         <child link="hand_link"/>
@@ -188,5 +188,5 @@
         <parent link="hand_link"/>
         <child link="tool_link"/>
-        <origin xyz="0 0 ${distance_hand_tool}" rpy="${-PI/2} ${-PI/2} 0"/>
+        <origin xyz="0 0 ${distance_hand_tool}" rpy="0 0 0"/>
     </joint>
     <!--

Commit message: fix: make sure ned2's urdf follow DH conventions

File: niryo_robot_description/urdf/ned2/niryo_ned2.urdf.xacro (robot description, xacro)
@@ -106,5 +106,5 @@
         </inertial>
         <visual>
-            <origin xyz="0 0 0" rpy="0 0 ${-PI/2}"/>
+            <origin xyz="0 0 0.065" rpy="0 0 ${-PI/2}"/>
             <geometry>
                 <mesh filename="package://niryo_robot_description/meshes/ned2/collada/forearm_link.dae"/>
@@ -160,5 +160,5 @@
         </inertial>
         <visual>
-            <origin xyz="0 0 0" rpy="0 0 ${-PI/2}"/>
+            <origin xyz="0 0 0.0197" rpy="0 0 ${-PI/2}"/>
             <geometry>
                 <mesh filename="package://niryo_robot_description/meshes/ned2/collada/hand_link.dae"/>
@@ -205,5 +205,5 @@
     </joint>
     <joint name="joint_4" type="revolute">
-        <origin xyz="0.0325 -0.065 0" rpy="${PI/2} 0 0"/>
+        <origin xyz="0.0325 0 0" rpy="${PI/2} 0 0"/>
         <parent link="elbow_link"/>
         <child link="forearm_link"/>
@@ -213,5 +213,5 @@
     </joint>
     <joint name="joint_5" type="revolute">
-        <origin xyz="0 0 0.17" rpy="${-PI/2} 0 0"/>
+        <origin xyz="0 0 0.235" rpy="${-PI/2} 0 0"/>
         <parent link="forearm_link"/>
         <child link="wrist_link"/>
@@ -221,5 +221,5 @@
     </joint>
     <joint name="joint_6" type="revolute">
-        <origin xyz="0.00925 -0.0197 0" rpy="${PI/2} 0 0"/>
+        <origin xyz="0.00925 0 0" rpy="${PI/2} 0 0"/>
         <parent link="wrist_link"/>
         <child link="hand_link"/>

Commit message: chore; revert unecessary changes in URDF

File: niryo_robot_description/urdf/ned2/niryo_ned2.urdf.xacro (robot description, xacro)
@@ -106,5 +106,5 @@
         </inertial>
         <visual>
-            <origin xyz="0 0 0.065" rpy="0 0 ${-PI/2}"/>
+            <origin xyz="0 0 0" rpy="0 0 ${-PI/2}"/>
             <geometry>
                 <mesh filename="package://niryo_robot_description/meshes/ned2/collada/forearm_link.dae"/>
@@ -160,5 +160,5 @@
         </inertial>
         <visual>
-            <origin xyz="0 0 0.0197" rpy="0 0 ${-PI/2}"/>
+            <origin xyz="0 0 0" rpy="0 0 ${-PI/2}"/>
             <geometry>
                 <mesh filename="package://niryo_robot_description/meshes/ned2/collada/hand_link.dae"/>
@@ -205,5 +205,5 @@
     </joint>
     <joint name="joint_4" type="revolute">
-        <origin xyz="0.0325 0 0" rpy="${PI/2} 0 0"/>
+        <origin xyz="0.0325 -0.065 0" rpy="${PI/2} 0 0"/>
         <parent link="elbow_link"/>
         <child link="forearm_link"/>
@@ -213,5 +213,5 @@
     </joint>
     <joint name="joint_5" type="revolute">
-        <origin xyz="0 0 0.235" rpy="${-PI/2} 0 0"/>
+        <origin xyz="0 0 0.17" rpy="${-PI/2} 0 0"/>
         <parent link="forearm_link"/>
         <child link="wrist_link"/>
@@ -221,5 +221,5 @@
     </joint>
     <joint name="joint_6" type="revolute">
-        <origin xyz="0.00925 0 0" rpy="${PI/2} 0 0"/>
+        <origin xyz="0.00925 -0.0197 0" rpy="${PI/2} 0 0"/>
         <parent link="wrist_link"/>
         <child link="hand_link"/>

Commit message: refactor: (SN-805) Rollback TCPv2

File: niryo_robot_description/urdf/ned2/niryo_ned2.urdf.xacro (robot description, xacro)
@@ -231,5 +231,5 @@
         <parent link="hand_link"/>
         <child link="tool_link"/>
-        <origin xyz="0 0 ${distance_hand_tool}" rpy="0 0 0"/>
+        <origin xyz="0 0 ${distance_hand_tool}" rpy="${PI} -${PI/2} 0"/>
     </joint>
     <!--

File: niryo_robot_description/urdf/ned2/without_mesh_niryo_ned2.urdf.xacro (robot description, xacro)
@@ -188,5 +188,5 @@
         <parent link="hand_link"/>
         <child link="tool_link"/>
-        <origin xyz="0 0 ${distance_hand_tool}" rpy="0 0 0"/>
+        <origin xyz="0 0 ${distance_hand_tool}" rpy="${PI} -${PI/2} 0"/>
     </joint>
     <!--

File: niryo_robot_description/urdf/ned3pro/niryo_ned3pro.urdf.xacro (robot description, xacro)
@@ -221,5 +221,5 @@
         <parent link="hand_link" />
         <child link="tool_link" />
-        <origin xyz="0 0 ${distance_hand_tool}" rpy="0 0 0" />
+        <origin xyz="0 0 ${distance_hand_tool}" rpy="${PI} -${PI/2} 0" />
     </joint>
     <joint name="joint_led_ring" type="fixed">

File: niryo_robot_description/urdf/ned3pro/without_mesh_niryo_ned3pro.urdf.xacro (robot description, xacro)
@@ -174,5 +174,5 @@
         <parent link="hand_link" />
         <child link="tool_link" />
-        <origin xyz="0 0 ${distance_hand_tool}" rpy="0 0 0" />
+        <origin xyz="0 0 ${distance_hand_tool}" rpy="${PI} -${PI/2} 0" />
     </joint>
     <joint name="joint_led_ring" type="fixed">
