Commit message: enhance joints limits on j5

File: niryo_robot_description/urdf/ned2/niryo_ned2_param.urdf.xacro (robot description, xacro)
@@ -13,6 +13,6 @@
     <xacro:property name="limit_low_forearm_rotation" value="-120.0"/>
     <xacro:property name="limit_up_forearm_rotation" value="120.0"/>
-    <xacro:property name="limit_low_wrist_rotation" value="-100.0"/>
-    <xacro:property name="limit_up_wrist_rotation" value="55.0"/>
+    <xacro:property name="limit_low_wrist_rotation" value="-110.0"/>
+    <xacro:property name="limit_up_wrist_rotation" value="110.0"/>
     <xacro:property name="limit_low_hand_rotation" value="-145.0"/>
     <xacro:property name="limit_up_hand_rotation" value="145.0"/>

Commit message: Fix vision

File: niryo_robot_description/urdf/ned2/niryo_ned2_param.urdf.xacro (robot description, xacro)
@@ -5,6 +5,6 @@
     <!-- Properties -->
     <xacro:property name="distance_hand_tool" value="0.0215"/>
-    <xacro:property name="limit_low_shoulder_rotation" value="-170.0"/>
-    <xacro:property name="limit_up_shoulder_rotation" value="170.0"/>
+    <xacro:property name="limit_low_shoulder_rotation" value="-169.0"/>
+    <xacro:property name="limit_up_shoulder_rotation" value="169.0"/>
     <xacro:property name="limit_low_arm_rotation" value="-120.0"/>
     <xacro:property name="limit_up_arm_rotation" value="35.0"/>

Commit message: [Bugfix] Fixed urdf ned2

File: niryo_robot_description/urdf/ned2/niryo_ned2_param.urdf.xacro (robot description, xacro)
@@ -14,5 +14,5 @@
     <xacro:property name="limit_up_forearm_rotation" value="119.75"/>
     <xacro:property name="limit_low_wrist_rotation" value="-110.01"/>
-    <xacro:property name="limit_up_wrist_rotation" value="60.17"/>
+    <xacro:property name="limit_up_wrist_rotation" value="110.0"/>
     <xacro:property name="limit_low_hand_rotation" value="-144.96"/>
     <xacro:property name="limit_up_hand_rotation" value="144.96"/>

Commit message: Fix Niryo one vision + tool + conveyor + add doc

File: niryo_robot_description/urdf/ned2/niryo_ned2_param.urdf.xacro (robot description, xacro)
@@ -14,5 +14,5 @@
     <xacro:property name="limit_up_forearm_rotation" value="119.75"/>
     <xacro:property name="limit_low_wrist_rotation" value="-110.01"/>
-    <xacro:property name="limit_up_wrist_rotation" value="110.0"/>
+    <xacro:property name="limit_up_wrist_rotation" value="110.17"/>
     <xacro:property name="limit_low_hand_rotation" value="-144.96"/>
     <xacro:property name="limit_up_hand_rotation" value="144.96"/>

File: niryo_robot_description/urdf/one/without_mesh_niryo_one.urdf.xacro (robot description, xacro)
@@ -64,5 +64,5 @@
         <origin xyz="${distance_elbow_forearm_x} ${distance_elbow_forearm_y} 0" rpy="0 ${PI/2} 0" />
 		<limit effort="1" velocity="1.0" lower="${(limit_low_forearm_rotation + safety_pos_margin) * deg_to_rad}"
-               upper="${(limit_up_forearm_rotation - safety_pos_margin) * deg_to_rad}" />
+               upper="${(limit_up_forearm_rotation - safety_pos_margin) * deg_to_rad }" />
 		<axis xyz="0 0 1" />
 	</joint>
@@ -72,5 +72,5 @@
 		<origin xyz="0 0 ${distance_forearm_wrist_z}" rpy="0 ${-PI/2} 0" />
 		<limit effort="1" velocity="1.0" lower="${(limit_low_wrist_rotation + safety_pos_margin) * deg_to_rad}"
-               upper="${(limit_up_wrist_rotation - safety_pos_margin) * deg_to_rad}" />
+               upper="${(limit_up_wrist_rotation - safety_pos_margin) * deg_to_rad }" />
 		<axis xyz="0 0 1" />
 	</joint>

Commit message: Release v4.0.0

File: niryo_robot_description/urdf/ned2/niryo_ned2_param.urdf.xacro (robot description, xacro)
@@ -14,5 +14,5 @@
     <xacro:property name="limit_up_forearm_rotation" value="119.75"/>
     <xacro:property name="limit_low_wrist_rotation" value="-110.01"/>
-    <xacro:property name="limit_up_wrist_rotation" value="60.17"/>
+    <xacro:property name="limit_up_wrist_rotation" value="110.17"/>
     <xacro:property name="limit_low_hand_rotation" value="-144.96"/>
     <xacro:property name="limit_up_hand_rotation" value="144.96"/>

Commit message: fix: correct feedback output in the move function

File: niryo_robot_description/urdf/ned2/niryo_ned2_param.urdf.xacro (robot description, xacro)
@@ -10,5 +10,5 @@
     <xacro:property name="limit_up_arm_rotation" value="34.96"/>
     <xacro:property name="limit_low_elbow_rotation" value="-76.78"/>
-    <xacro:property name="limit_up_elbow_rotation" value="89.96"/>
+    <xacro:property name="limit_up_elbow_rotation" value="85.5"/>
     <xacro:property name="limit_low_forearm_rotation" value="-119.75"/>
     <xacro:property name="limit_up_forearm_rotation" value="119.75"/>
