Commit message: Stack v5.5.0

File: niryo_robot_description/urdf/ned3pro/niryo_ned3pro.transmission.xacro (robot description, xacro)
@@ -1,4 +1,4 @@
 <?xml version="1.0"?>
-<robot xmlns:xacro="http://ros.org/wiki/xacro"  name="niryo_ned3">
+<robot xmlns:xacro="http://ros.org/wiki/xacro"  name="niryo_ned3pro">
   <!-- Transmission macro -->
   <xacro:macro name="SimpleTransmissionPosition" params="joint n">

File: niryo_robot_description/urdf/ned3pro/niryo_ned3pro.urdf.xacro (robot description, xacro)
@@ -1,6 +1,6 @@
 <?xml version="1.0"?>
-<robot xmlns:xacro="http://www.ros.org/wiki/xacro" name="niryo_ned3">
+<robot xmlns:xacro="http://www.ros.org/wiki/xacro" name="niryo_ned3pro">
     <!-- Import Properties -->
-    <xacro:include filename="$(find niryo_robot_description)/urdf/ned3/niryo_ned3_param.urdf.xacro" />
+    <xacro:include filename="$(find niryo_robot_description)/urdf/ned3pro/niryo_ned3pro_param.urdf.xacro" />
     <!-- Links -->
     <link name="world" />
@@ -12,8 +12,14 @@
                 izz="0.0254462446" />
         </inertial>
-        <collision>
-            <origin xyz="0 0 0" rpy="0 0 0" />
-            <geometry>
-                <mesh filename="package://niryo_robot_description/meshes/ned3/stl/base_link.STL" />
+        <visual>
+            <origin xyz="0 0 0" rpy="0 0 0" />
+            <geometry>
+                <mesh filename="package://niryo_robot_description/meshes/ned3pro/stl/base_link.STL" />
+            </geometry>
+        </visual>
+        <collision>
+            <origin xyz="0 0 0" rpy="0 0 0" />
+            <geometry>
+                <mesh filename="package://niryo_robot_description/meshes/ned3pro/stl/base_link.STL" />
             </geometry>
         </collision>
@@ -28,8 +34,15 @@
                 izz="0.00292927208" />
         </inertial>
-        <collision>
-            <origin xyz="0 0 0" rpy="0 0 0" />
-            <geometry>
-                <mesh filename="package://niryo_robot_description/meshes/ned3/stl/shoulder_link.STL" />
+        <visual>
+            <origin xyz="0 0 0" rpy="0 0 0" />
+            <geometry>
+                <mesh
+                    filename="package://niryo_robot_description/meshes/ned3pro/stl/shoulder_link.STL" />
+            </geometry>
+        </visual>
+        <collision>
+            <origin xyz="0 0 0" rpy="0 0 0" />
+            <geometry>
+                <mesh filename="package://niryo_robot_description/meshes/ned3pro/stl/shoulder_link.STL" />
             </geometry>
         </collision>
@@ -42,8 +55,14 @@
                 izz="0.00879836087" />
         </inertial>
-        <collision>
+        <visual>
             <origin xyz="0 0 0" rpy="0 0 ${PI}" />
             <geometry>
-                <mesh filename="package://niryo_robot_description/meshes/ned3/stl/arm_link.STL" />
+                <mesh filename="package://niryo_robot_description/meshes/ned3pro/stl/arm_link.STL" />
+            </geometry>
+        </visual>
+        <collision>
+            <origin xyz="0 0 0" rpy="0 0 ${PI}" />
+            <geometry>
+                <mesh filename="package://niryo_robot_description/meshes/ned3pro/stl/arm_link.STL" />
             </geometry>
         </collision>
@@ -56,8 +75,15 @@
                 izz="0.00043216299" />
         </inertial>
-        <collision>
+        <visual>
             <origin xyz="0 0 0" rpy="${PI} 0 ${-PI/2}" />
             <geometry>
-                <mesh filename="package://niryo_robot_description/meshes/ned3/stl/elbow_link.STL" />
+                <mesh
+                    filename="package://niryo_robot_description/meshes/ned3pro/stl/elbow_link.STL" />
+            </geometry>
+        </visual>
+        <collision>
+            <origin xyz="0 0 0" rpy="${PI} 0 ${-PI/2}" />
+            <geometry>
+                <mesh filename="package://niryo_robot_description/meshes/ned3pro/stl/elbow_link.STL" />
             </geometry>
         </collision>
@@ -70,8 +96,15 @@
                 izz="0.00029473313" />
         </inertial>
-        <collision>
+        <visual>
             <origin xyz="0 0 0" rpy="${PI} 0 0" />
             <geometry>
-                <mesh filename="package://niryo_robot_description/meshes/ned3/stl/forearm_link.STL" />
+                <mesh
+                    filename="package://niryo_robot_description/meshes/ned3pro/stl/forearm_link.STL" />
+            </geometry>
+        </visual>
+        <collision>
+            <origin xyz="0 0 0" rpy="${PI} 0 0" />
+            <geometry>
+                <mesh filename="package://niryo_robot_description/meshes/ned3pro/stl/forearm_link.STL" />
             </geometry>
         </collision>
@@ -84,9 +117,17 @@
                 izz="0.00019643162" />
         </inertial>
-        <collision>
+        <visual>
             <origin xyz="0 0 0"
                 rpy="0 0 ${PI/2}" />
             <geometry>
-                <mesh filename="package://niryo_robot_description/meshes/ned3/stl/wrist_link.STL" />
+                <mesh
+                    filename="package://niryo_robot_description/meshes/ned3pro/stl/wrist_link.STL" />
+            </geometry>
+        </visual>
+        <collision>
+            <origin xyz="0 0 0"
+                rpy="0 0 ${PI/2}" />
+            <geometry>
+                <mesh filename="package://niryo_robot_description/meshes/ned3pro/stl/wrist_link.STL" />
             </geometry>
         </collision>
@@ -99,8 +140,14 @@
                 izz="0.00000040812" />
         </inertial>
-        <collision>
-            <origin xyz="0 0 0" rpy="0 0 0" />
-            <geometry>
-                <mesh filename="package://niryo_robot_description/meshes/ned3/stl/hand_link.STL" />
+        <visual>
+            <origin xyz="0 0 0" rpy="0 0 0" />
+            <geometry>
+                <mesh filename="package://niryo_robot_description/meshes/ned3pro/stl/hand_link.STL" />
+            </geometry>
+        </visual>
+        <collision>
+            <origin xyz="0 0 0" rpy="0 0 0" />
+            <geometry>
+                <mesh filename="package://niryo_robot_description/meshes/ned3pro/stl/hand_link.STL" />
             </geometry>
         </collision>

File: niryo_robot_description/urdf/ned3pro/niryo_ned3pro_camera.urdf.xacro (robot description, xacro)
@@ -1,6 +1,6 @@
 <?xml version="1.0"?>
-<robot xmlns:xacro="http://www.ros.org/wiki/xacro" name="niryo_ned3">
+<robot xmlns:xacro="http://www.ros.org/wiki/xacro" name="niryo_ned3pro">
     <!-- Including base robot -->
-    <xacro:include filename="$(find niryo_robot_description)/urdf/ned3/niryo_ned3_gazebo.urdf.xacro"/>
+    <xacro:include filename="$(find niryo_robot_description)/urdf/ned3pro/niryo_ned3pro_gazebo.urdf.xacro"/>
     <!-- Properties -->
     <xacro:property name="cameraWidth" value="0.01"/>

File: niryo_robot_description/urdf/ned3pro/niryo_ned3pro_gazebo.urdf.xacro (robot description, xacro)
@@ -1,4 +1,4 @@
 <?xml version="1.0"?>
-<robot xmlns:xacro="http://www.ros.org/wiki/xacro" name="niryo_ned3">
+<robot xmlns:xacro="http://www.ros.org/wiki/xacro" name="niryo_ned3pro">
     <!-- Enable Gazebo control-->
     <gazebo>
@@ -8,6 +8,6 @@
     </gazebo>
     <!-- Import Robot -->
-    <xacro:include filename="$(find niryo_robot_description)/urdf/ned3/niryo_ned3.urdf.xacro"/>
+    <xacro:include filename="$(find niryo_robot_description)/urdf/ned3pro/niryo_ned3pro.urdf.xacro"/>
     <!-- Import Transmission -->
-    <xacro:include filename="$(find niryo_robot_description)/urdf/ned3/niryo_ned3.transmission.xacro"/>
+    <xacro:include filename="$(find niryo_robot_description)/urdf/ned3pro/niryo_ned3pro.transmission.xacro"/>
 </robot>

File: niryo_robot_description/urdf/ned3pro/niryo_ned3pro_gripper1_n_camera.urdf.xacro (robot description, xacro)
@@ -1,5 +1,5 @@
 <?xml version="1.0"?>
-<robot xmlns:xacro="http://www.ros.org/wiki/xacro" name="niryo_ned3">
-    <xacro:include filename="$(find niryo_robot_description)/urdf/ned3/niryo_ned3_camera.urdf.xacro"/>
+<robot xmlns:xacro="http://www.ros.org/wiki/xacro" name="niryo_ned3pro">
+    <xacro:include filename="$(find niryo_robot_description)/urdf/ned3pro/niryo_ned3pro_camera.urdf.xacro"/>
     <!-- gazebo joint state publisher for all joints. Necessary to control mors -->
     <gazebo>

File: niryo_robot_description/urdf/ned3pro/niryo_ned3pro_param.urdf.xacro (robot description, xacro)
@@ -1,4 +1,4 @@
 <?xml version="1.0"?>
-<robot xmlns:xacro="http://www.ros.org/wiki/xacro" name="niryo_ned3">
+<robot xmlns:xacro="http://www.ros.org/wiki/xacro" name="niryo_ned3pro">
     <xacro:property name="PI" value="3.14159265359"/>
     <!-- Properties -->

File: niryo_robot_description/urdf/ned3pro/without_mesh_niryo_ned3pro.urdf.xacro (robot description, xacro)
@@ -1,6 +1,6 @@
 <?xml version="1.0"?>
-<robot xmlns:xacro="http://www.ros.org/wiki/xacro" name="niryo_ned3">
+<robot xmlns:xacro="http://www.ros.org/wiki/xacro" name="niryo_ned3pro">
     <!-- Import Properties -->
-    <xacro:include filename="$(find niryo_robot_description)/urdf/ned3/niryo_ned3_param.urdf.xacro" />
+    <xacro:include filename="$(find niryo_robot_description)/urdf/ned3pro/niryo_ned3pro_param.urdf.xacro" />
     <!-- Links -->
     <link name="world" />
@@ -12,14 +12,8 @@
                 izz="0.0254462446" />
         </inertial>
-        <visual>
-            <origin xyz="0 0 0" rpy="0 0 0" />
-            <geometry>
-                <mesh filename="package://niryo_robot_description/meshes/ned3/stl/base_link.STL" />
-            </geometry>
-        </visual>
         <collision>
             <origin xyz="0 0 0" rpy="0 0 0" />
             <geometry>
-                <mesh filename="package://niryo_robot_description/meshes/ned3/stl/base_link.STL" />
+                <mesh filename="package://niryo_robot_description/meshes/ned3pro/stl/base_link.STL" />
             </geometry>
         </collision>
@@ -34,15 +28,8 @@
                 izz="0.00292927208" />
         </inertial>
-        <visual>
-            <origin xyz="0 0 0" rpy="0 0 0" />
-            <geometry>
-                <mesh
-                    filename="package://niryo_robot_description/meshes/ned3/stl/shoulder_link.STL" />
-            </geometry>
-        </visual>
         <collision>
             <origin xyz="0 0 0" rpy="0 0 0" />
             <geometry>
-                <mesh filename="package://niryo_robot_description/meshes/ned3/stl/shoulder_link.STL" />
+                <mesh filename="package://niryo_robot_description/meshes/ned3pro/stl/shoulder_link.STL" />
             </geometry>
         </collision>
@@ -55,14 +42,8 @@
                 izz="0.00879836087" />
         </inertial>
-        <visual>
-            <origin xyz="0 0 0" rpy="0 0 ${PI}" />
-            <geometry>
-                <mesh filename="package://niryo_robot_description/meshes/ned3/stl/arm_link.STL" />
-            </geometry>
-        </visual>
         <collision>
             <origin xyz="0 0 0" rpy="0 0 ${PI}" />
             <geometry>
-                <mesh filename="package://niryo_robot_description/meshes/ned3/stl/arm_link.STL" />
+                <mesh filename="package://niryo_robot_description/meshes/ned3pro/stl/arm_link.STL" />
             </geometry>
         </collision>
@@ -75,15 +56,8 @@
                 izz="0.00043216299" />
         </inertial>
-        <visual>
-            <origin xyz="0 0 0" rpy="${PI} 0 ${-PI/2}" />
-            <geometry>
-                <mesh
-                    filename="package://niryo_robot_description/meshes/ned3/stl/elbow_link.STL" />
-            </geometry>
-        </visual>
         <collision>
             <origin xyz="0 0 0" rpy="${PI} 0 ${-PI/2}" />
             <geometry>
-                <mesh filename="package://niryo_robot_description/meshes/ned3/stl/elbow_link.STL" />
+                <mesh filename="package://niryo_robot_description/meshes/ned3pro/stl/elbow_link.STL" />
             </geometry>
         </collision>
@@ -96,15 +70,8 @@
                 izz="0.00029473313" />
         </inertial>
-        <visual>
-            <origin xyz="0 0 0" rpy="${PI} 0 0" />
-            <geometry>
-                <mesh
-                    filename="package://niryo_robot_description/meshes/ned3/stl/forearm_link.STL" />
-            </geometry>
-        </visual>
         <collision>
             <origin xyz="0 0 0" rpy="${PI} 0 0" />
             <geometry>
-                <mesh filename="package://niryo_robot_description/meshes/ned3/stl/forearm_link.STL" />
+                <mesh filename="package://niryo_robot_description/meshes/ned3pro/stl/forearm_link.STL" />
             </geometry>
         </collision>
@@ -117,17 +84,9 @@
                 izz="0.00019643162" />
         </inertial>
-        <visual>
-            <origin xyz="0 0 0"
-                rpy="0 0 ${PI/2}" />
-            <geometry>
-                <mesh
-                    filename="package://niryo_robot_description/meshes/ned3/stl/wrist_link.STL" />
-            </geometry>
-        </visual>
         <collision>
             <origin xyz="0 0 0"
                 rpy="0 0 ${PI/2}" />
             <geometry>
-                <mesh filename="package://niryo_robot_description/meshes/ned3/stl/wrist_link.STL" />
+                <mesh filename="package://niryo_robot_description/meshes/ned3pro/stl/wrist_link.STL" />
             </geometry>
         </collision>
@@ -140,14 +99,8 @@
                 izz="0.00000040812" />
         </inertial>
-        <visual>
-            <origin xyz="0 0 0" rpy="0 0 0" />
-            <geometry>
-                <mesh filename="package://niryo_robot_description/meshes/ned3/stl/hand_link.STL" />
-            </geometry>
-        </visual>
         <collision>
             <origin xyz="0 0 0" rpy="0 0 0" />
             <geometry>
-                <mesh filename="package://niryo_robot_description/meshes/ned3/stl/hand_link.STL" />
+                <mesh filename="package://niryo_robot_description/meshes/ned3pro/stl/hand_link.STL" />
             </geometry>
         </collision>
