Commit message: fix: Wrong tf in Ned3 pro URDF

File: niryo_robot_description/urdf/ned3pro/niryo_ned3pro.urdf.xacro (robot description, xacro)
@@ -182,5 +182,5 @@
     </joint>
     <joint name="joint_3" type="revolute">
-        <origin xyz="0 0.23061 0" rpy="0 0 ${PI/2}" />
+        <origin xyz="0.12 0.23031 0" rpy="0 0 ${PI/2}" />
         <parent link="arm_link" />
         <child link="elbow_link" />

Commit message: fix: Wrong tf in Ned3 pro URDF

File: niryo_robot_description/urdf/ned3pro/niryo_ned3pro.urdf.xacro (robot description, xacro)
@@ -182,5 +182,5 @@
     </joint>
     <joint name="joint_3" type="revolute">
-        <origin xyz="0.12 0.23031 0" rpy="0 0 ${PI/2}" />
+        <origin xyz="0.012 0.23031 0" rpy="0 0 ${PI/2}" />
         <parent link="arm_link" />
         <child link="elbow_link" />

Commit message: fix: wrong tf in ned3pro URDF

File: niryo_robot_description/urdf/ned3pro/niryo_ned3pro.urdf.xacro (robot description, xacro)
@@ -201,5 +201,5 @@
     </joint>
     <joint name="joint_5" type="revolute">
-        <origin xyz="0 0 0.23975" rpy="${-PI/2} 0 0" />
+        <origin xyz="0 0 0.22975" rpy="${-PI/2} 0 0" />
         <parent link="forearm_link" />
         <child link="wrist_link" />

File: niryo_robot_description/urdf/ned3pro/without_mesh_niryo_ned3pro.urdf.xacro (robot description, xacro)
@@ -135,5 +135,5 @@
     </joint>
     <joint name="joint_3" type="revolute">
-        <origin xyz="0 0.23061 0" rpy="0 0 ${PI/2}" />
+        <origin xyz="0.012 0.23031 0" rpy="0 0 ${PI/2}" />
         <parent link="arm_link" />
         <child link="elbow_link" />
@@ -154,5 +154,5 @@
     </joint>
     <joint name="joint_5" type="revolute">
-        <origin xyz="0 0 0.23975" rpy="${-PI/2} 0 0" />
+        <origin xyz="0 0 0.22975" rpy="${-PI/2} 0 0" />
         <parent link="forearm_link" />
         <child link="wrist_link" />

Commit message: fix: tools transform

File: niryo_robot_description/urdf/ned3pro/niryo_ned3pro.urdf.xacro (robot description, xacro)
@@ -201,5 +201,5 @@
     </joint>
     <joint name="joint_5" type="revolute">
-        <origin xyz="0 0 0.22975" rpy="${-PI/2} 0 0" />
+        <origin xyz="0 0 0.23975" rpy="${-PI/2} 0 0" />
         <parent link="forearm_link" />
         <child link="wrist_link" />

File: niryo_robot_description/urdf/ned3pro/without_mesh_niryo_ned3pro.urdf.xacro (robot description, xacro)
@@ -154,5 +154,5 @@
     </joint>
     <joint name="joint_5" type="revolute">
-        <origin xyz="0 0 0.22975" rpy="${-PI/2} 0 0" />
+        <origin xyz="0 0 0.23975" rpy="${-PI/2} 0 0" />
         <parent link="forearm_link" />
         <child link="wrist_link" />
